File: cameras_module.sch (KiCad schematic (older format))
At the start: 0 parts

Commit message: Creating schemas for camera FFC, connecting related pins to SoM, schema of I2C MUX and voltage transceiver; Adding RESET to power supplies; connecting to SoM 1v8 power output
Parts:
- added C?: C_100n_0402, antmicro-footprints:0402-cap, symbol antmicroCapacitors0402:C_100n_0402
- added J?: WE_68715014522, antmicro-footprints:WE_68715014522, symbol antmicroFCCConnectors:WE_68715014522
- added R? (x6): R_0R_0402, antmicro-footprints:0402-res, symbol antmicroResistors0402:R_0R_0402
- added R? (x9): R_2k_0402, antmicro-footprints:0402-res, symbol antmicroResistors0402:R_2k_0402
- added U?: PCA9547BS, antmicro-footprints:VQFN-24, symbol antmicroLogicSignalSwitchesMultiplexersDecoders:PCA9547BS
- added U?: NTS0102DP, antmicro-footprints:TSSOP-8_W3mm, symbol antmicroLogicTranslatorsLevelShifters:NTS0102DP
Connections:
- net labels added: 1V8_SOM, 3V3_CAM, 3V3_SYS, 5V0_SYS, CAM0_SCL, CAM0_SDA, CAM1_DATA, CAM1_SCL, CAM1_SDA, CAM2_DATA, CAM_I2C_SCL, CAM_I2C_SCL_MUX, CAM_I2C_SDA, CAM_I2C_SDA_MUX, CSI_0_CLK_N, CSI_0_CLK_P, CSI_0_LN0_N, CSI_0_LN0_P, CSI_0_LN1_N, CSI_0_LN1_P, CSI_0_LN2_N, CSI_0_LN2_P, CSI_0_LN3_N, CSI_0_LN3_P, CSI_1_CLK_N, CSI_1_CLK_P, CSI_1_LN0_N, CSI_1_LN0_P, CSI_1_LN1_N, CSI_1_LN1_P, CSI_1_LN2_N, CSI_1_LN2_P, CSI_1_LN3_N, CSI_1_LN3_P, GND, VSYNC_CAM1, VSYNC_CAM2
- wire segments 0 -> 117
- no-connect marks 0 -> 27
Other:
- note added: "Camera FFC\n\n"
- note added: "Camera I2C multiplexer\n"
- note added: "SoM to I2C Mux voltage translating transceiver"

Commit message: Creating schema for SD card connection
Connections:
- net labels added: LDO6_1P8
- net labels removed: 1V8_SOM
Changed lines of the file:
@@
 	4300 8500 4100 8500
 Text GLabel 2050 8000 0    50   Input ~ 0
-1V8_SOM
+LDO6_1P8
 Wire Wire Line
 	2050 8000 2350 8000

Commit message: Added annotations. Move to loclib
Parts:
- C33: renamed from C?; footprint antmicro-footprints:0402-cap -> sc606-baseboard-footprints:0402-cap; symbol antmicroCapacitors0402:C_100n_0402 -> sc606-baseboard:C_100n_0402
- J3: renamed from J?; footprint antmicro-footprints:WE_68715014522 -> sc606-baseboard-footprints:WE_68715014522; symbol antmicroFCCConnectors:WE_68715014522 -> sc606-baseboard:WE_68715014522
- R16, R17, R18, R19, R20, R27, R28, R29, R30: renamed from R?; footprint antmicro-footprints:0402-res -> sc606-baseboard-footprints:0402-res; symbol antmicroResistors0402:R_2k_0402 -> sc606-baseboard:R_2k_0402
- R21, R22, R23, R24, R25, R26: renamed from R?; footprint antmicro-footprints:0402-res -> sc606-baseboard-footprints:0402-res; symbol antmicroResistors0402:R_0R_0402 -> sc606-baseboard:R_0R_0402
- U3: renamed from U?; footprint antmicro-footprints:TSSOP-8_W3mm -> sc606-baseboard-footprints:TSSOP-8_W3mm; symbol antmicroLogicTranslatorsLevelShifters:NTS0102DP -> sc606-baseboard:NTS0102DP
- U4: renamed from U?; footprint antmicro-footprints:VQFN-24 -> sc606-baseboard-footprints:VQFN-24; symbol antmicroLogicSignalSwitchesMultiplexersDecoders:PCA9547BS -> sc606-baseboard:PCA9547BS
Changed lines of the file:
@@
 Camera I2C multiplexer\n
 $Comp
-L antmicroLogicSignalSwitchesMultiplexersDecoders:PCA9547BS U?
+L sc606-baseboard:PCA9547BS U4
 U 1 1 61E56C5B
 P 4950 4700
-F 0 "U?" H 4850 6089 60  0000 C CNN
+F 0 "U4" H 4850 6089 60  0000 C CNN
 F 1 "PCA9547BS" H 4850 5983 60  0000 C CNN
-F 2 "antmicro-footprints:VQFN-24" H 4700 3300 60  0001 C CNN
+F 2 "sc606-baseboard-footprints:VQFN-24" H 4700 3300 60  0001 C CNN
 F 3 "https://www.nxp.com/docs/en/data-sheet/PCA9547.pdf" H 4950 4700 60  0001 C CNN
 F 4 " NXP" H 4950 4700 50  0001 C CNN "Manufacturer"
@@
 $EndComp
 $Comp
-L antmicroCapacitors0402:C_100n_0402 C?
+L sc606-baseboard:C_100n_0402 C33
 U 1 1 61E589C6
 P 4000 5100
-F 0 "C?" H 4115 5145 60  0000 L CNN
+F 0 "C33" H 4115 5145 60  0000 L CNN
 F 1 "C_100n_0402" H 4000 4950 60  0001 C CNN
-F 2 "antmicro-footprints:0402-cap" H 4200 5300 60  0001 L CNN
+F 2 "sc606-baseboard-footprints:0402-cap" H 4200 5300 60  0001 L CNN
 F 3 "" H 4000 5100 50  0001 C CNN
 F 4 "Walsin" H 4200 5500 60  0001 L CNN "Manufacturer"
@@
 	4000 3600 4000 4950
 $Comp
-L power:GND #PWR?
+L sc606-baseboard:GND #PWR042
 U 1 1 61E5F2B7
 P 4000 6350
-F 0 "#PWR?" H 4000 6100 50  0001 C CNN
+F 0 "#PWR042" H 4000 6100 50  0001 C CNN
 F 1 "GND" H 4005 6177 50  0000 C CNN
 F 2 "" H 4000 6350 50  0001 C CNN
@@
 	3250 3900 2050 3900
 $Comp
-L antmicroResistors0402:R_0R_0402 R?
+L sc606-baseboard:R_0R_0402 R21
 U 1 1 61E63E68
 P 3700 3800
-F 0 "R?" H 3700 4013 60  0000 C CNN
+F 0 "R21" H 3700 4013 60  0000 C CNN
 F 1 "R_0R_0402" H 3700 3650 60  0001 C CNN
-F 2 "antmicro-footprints:0402-res" H 3900 4000 60  0001 L CNN
+F 2 "sc606-baseboard-footprints:0402-res" H 3900 4000 60  0001 L CNN
 F 3 "" H 3700 3800 50  0001 C CNN
 F 4 "PANASONIC" H 3900 4200 60  0001 L CNN "Manufacturer"
@@
 	3850 3800 4450 3800
 $Comp
-L antmicroResistors0402:R_0R_0402 R?
+L sc606-baseboard:R_0R_0402 R22
 U 1 1 61E641DF
 P 3700 3900
-F 0 "R?" H 3700 3777 60  0000 C CNN
+F 0 "R22" H 3700 3777 60  0000 C CNN
 F 1 "R_0R_0402" H 3700 3750 60  0001 C CNN
-F 2 "antmicro-footprints:0402-res" H 3900 4100 60  0001 L CNN
+F 2 "sc606-baseboard-footprints:0402-res" H 3900 4100 60  0001 L CNN
 F 3 "" H 3700 3900 50  0001 C CNN
 F 4 "PANASONIC" H 3900 4300 60  0001 L CNN "Manufacturer"
@@
 	2950 3400 3250 3400
 $Comp
-L antmicroResistors0402:R_2k_0402 R?
+L sc606-baseboard:R_2k_0402 R19
 U 1 1 61E68958
 P 2950 3550
-F 0 "R?" V 2905 3620 60  0000 L CNN
+F 0 "R19" V 2905 3620 60  0000 L CNN
 F 1 "R_2k_0402" H 2950 3400 60  0001 C CNN
-F 2 "antmicro-footprints:0402-res" H 3150 3750 60  0001 L CNN
+F 2 "sc606-baseboard-footprints:0402-res" H 3150 3750 60  0001 L CNN
 F 3 "" H 2950 3550 50  0001 C CNN
 F 4 "VISHAY" H 3150 3950 60  0001 L CNN "Manufacturer"
@@
 $EndComp
 $Comp
-L antmicroResistors0402:R_2k_0402 R?
+L sc606-baseboard:R_2k_0402 R20
 U 1 1 61E68DEE
 P 3250 3550
-F 0 "R?" V 3205 3620 60  0000 L CNN
+F 0 "R20" V 3205 3620 60  0000 L CNN
 F 1 "R_2k_0402" H 3250 3400 60  0001 C CNN
-F 2 "antmicro-footprints:0402-res" H 3450 3750 60  0001 L CNN
+F 2 "sc606-baseboard-footprints:0402-res" H 3450 3750 60  0001 L CNN
 F 3 "" H 3250 3550 50  0001 C CNN
 F 4 "VISHAY" H 3450 3950 60  0001 L CNN "Manufacturer"
@@
 	4450 4500 4450 5800
 $Comp
-L antmicroResistors0402:R_0R_0402 R?
+L sc606-baseboard:R_0R_0402 R23
 U 1 1 61E6A5CA
 P 6150 3600
-F 0 "R?" H 6350 3650 60  0000 C CNN
+F 0 "R23" H 6350 3650 60  0000 C CNN
 F 1 "R_0R_0402" H 6150 3450 60  0001 C CNN
-F 2 "antmicro-footprints:0402-res" H 6350 3800 60  0001 L CNN
+F 2 "sc606-baseboard-footprints:0402-res" H 6350 3800 60  0001 L CNN
 F 3 "" H 6150 3600 50  0001 C CNN
 F 4 "PANASONIC" H 6350 4000 60  0001 L CNN "Manufacturer"
@@
 $EndComp
 $Comp
-L antmicroResistors0402:R_0R_0402 R?
+L sc606-baseboard:R_0R_0402 R24
 U 1 1 61E6AAD1
 P 6150 3700
-F 0 "R?" H 6350 3750 60  0000 C CNN
+F 0 "R24" H 6350 3750 60  0000 C CNN
 F 1 "R_0R_0402" H 6150 3550 60  0001 C CNN
-F 2 "antmicro-footprints:0402-res" H 6350 3900 60  0001 L CNN
+F 2 "sc606-baseboard-footprints:0402-res" H 6350 3900 60  0001 L CNN
 F 3 "" H 6150 3700 50  0001 C CNN
 F 4 "PANASONIC" H 6350 4100 60  0001 L CNN "Manufacturer"
@@
 $EndComp
 $Comp
-L antmicroResistors0402:R_0R_0402 R?
+L sc606-baseboard:R_0R_0402 R25
 U 1 1 61E6AE4A
 P 6150 3900
-F 0 "R?" H 6350 3950 60  0000 C CNN
+F 0 "R25" H 6350 3950 60  0000 C CNN
 F 1 "R_0R_0402" H 6150 3750 60  0001 C CNN
-F 2 "antmicro-footprints:0402-res" H 6350 4100 60  0001 L CNN
+F 2 "sc606-baseboard-footprints:0402-res" H 6350 4100 60  0001 L CNN
 F 3 "" H 6150 3900 50  0001 C CNN
 F 4 "PANASONIC" H 6350 4300 60  0001 L CNN "Manufacturer"
@@
 $EndComp
 $Comp
-L antmicroResistors0402:R_0R_0402 R?
+L sc606-baseboard:R_0R_0402 R26
 U 1 1 61E6B0E9
 P 6150 4000
-F 0 "R?" H 6350 4050 60  0000 C CNN
+F 0 "R26" H 6350 4050 60  0000 C CNN
 F 1 "R_0R_0402" H 6150 3850 60  0001 C CNN
-F 2 "antmicro-footprints:0402-res" H 6350 4200 60  0001 L CNN
+F 2 "sc606-baseboard-footprints:0402-res" H 6350 4200 60  0001 L CNN
 F 3 "" H 6150 4000 50  0001 C CNN
 F 4 "PANASONIC" H 6350 4400 60  0001 L CNN "Manufacturer"
@@
 Camera FFC\n\n
 $Comp
-L antmicroFCCConnectors:WE_68715014522 J?
+L sc606-baseboard:WE_68715014522 J3
 U 1 1 61E964B1
 P 12800 3900
-F 0 "J?" H 12880 3092 50  0000 L CNN
+F 0 "J3" H 12880 3092 50  0000 L CNN
 F 1 "WE_68715014522" H 12880 3001 50  0000 L CNN
-F 2 "antmicro-footprints:WE_68715014522" H 12600 350 50  0001 C CNN
+F 2 "sc606-baseboard-footprints:WE_68715014522" H 12600 350 50  0001 C CNN
 F 3 "https://katalog.we-online.de/em/datasheet/6871xx14522.pdf" H 12800 250 50  0001 C CNN
 F 4 "68715014522 " H 13200 3300 60  0001 L CNN "MPN"
@@
 	12600 6400 10900 6400
 $Comp
-L antmicroResistors0402:R_2k_0402 R?
+L sc606-baseboard:R_2k_0402 R27
 U 1 1 61EAFCF7
 P 10300 5450
-F 0 "R?" H 10250 5350 60  0000 L CNN
+F 0 "R27" H 10250 5350 60  0000 L CNN
 F 1 "R_2k_0402" H 10300 5300 60  0001 C CNN
-F 2 "antmicro-footprints:0402-res" H 10500 5650 60  0001 L CNN
+F 2 "sc606-baseboard-footprints:0402-res" H 10500 5650 60  0001 L CNN
 F 3 "" H 10300 5450 50  0001 C CNN
 F 4 "VISHAY" H 10500 5850 60  0001 L CNN "Manufacturer"
@@
 $EndComp
 $Comp
-L antmicroResistors0402:R_2k_0402 R?
+L sc606-baseboard:R_2k_0402 R28
 U 1 1 61EB041B
 P 10500 5450
-F 0 "R?" H 10450 5350 60  0000 L CNN
+F 0 "R28" H 10450 5350 60  0000 L CNN
 F 1 "R_2k_0402" H 10500 5300 60  0001 C CNN
-F 2 "antmicro-footprints:0402-res" H 10700 5650 60  0001 L CNN
+F 2 "sc606-baseboard-footprints:0402-res" H 10700 5650 60  0001 L CNN
 F 3 "" H 10500 5450 50  0001 C CNN
 F 4 "VISHAY" H 10700 5850 60  0001 L CNN "Manufacturer"
@@
 $EndComp
 $Comp
-L antmicroResistors0402:R_2k_0402 R?
+L sc606-baseboard:R_2k_0402 R29
 U 1 1 61EB08C8
 P 10700 5450
-F 0 "R?" H 10650 5350 60  0000 L CNN
+F 0 "R29" H 10650 5350 60  0000 L CNN
 F 1 "R_2k_0402" H 10700 5300 60  0001 C CNN
-F 2 "antmicro-footprints:0402-res" H 10900 5650 60  0001 L CNN
+F 2 "sc606-baseboard-footprints:0402-res" H 10900 5650 60  0001 L CNN
 F 3 "" H 10700 5450 50  0001 C CNN
 F 4 "VISHAY" H 10900 5850 60  0001 L CNN "Manufacturer"
@@
 $EndComp
 $Comp
-L antmicroResistors0402:R_2k_0402 R?
+L sc606-baseboard:R_2k_0402 R30
 U 1 1 61EB0CC5
 P 10900 5450
-F 0 "R?" H 10850 5350 60  0000 L CNN
+F 0 "R30" H 10850 5350 60  0000 L CNN
 F 1 "R_2k_0402" H 10900 5300 60  0001 C CNN
-F 2 "antmicro-footprints:0402-res" H 11100 5650 60  0001 L CNN
+F 2 "sc606-baseboard-footprints:0402-res" H 11100 5650 60  0001 L CNN
 F 3 "" H 10900 5450 50  0001 C CNN
 F 4 "VISHAY" H 11100 5850 60  0001 L CNN "Manufacturer"
@@
 CAM_I2C_SCL_MUX
 $Comp
-L antmicroLogicTranslatorsLevelShifters:NTS0102DP U?
+L sc606-baseboard:NTS0102DP U3
 U 1 1 61EE57DC
 P 3700 8750
-F 0 "U?" H 3700 9265 50  0000 C CNN
+F 0 "U3" H 3700 9265 50  0000 C CNN
 F 1 "NTS0102DP" H 3700 9174 50  0000 C CNN
-F 2 "antmicro-footprints:TSSOP-8_W3mm" H 3600 9250 50  0001 C CNN
+F 2 "sc606-baseboard-footprints:TSSOP-8_W3mm" H 3600 9250 50  0001 C CNN
 F 3 "" H 4350 9500 50  0001 C CNN
 F 4 "NTS0102DP" H 3650 8350 50  0001 C CNN "MPN"
@@
 $EndComp
 $Comp
-L power:GND #PWR?
+L sc606-baseboard:GND #PWR043
 U 1 1 61EE63E6
 P 4100 9000
-F 0 "#PWR?" H 4100 8750 50  0001 C CNN
+F 0 "#PWR043" H 4100 8750 50  0001 C CNN
 F 1 "GND" H 4105 8827 50  0000 C CNN
 F 2 "" H 4100 9000 50  0001 C CNN
@@
 	2900 8800 3300 8800
 $Comp
-L antmicroResistors0402:R_2k_0402 R?
+L sc606-baseboard:R_2k_0402 R18
 U 1 1 61FFF734
 P 2900 8250
-F 0 "R?" V 2950 8450 60  0000 R CNN
+F 0 "R18" V 2950 8450 60  0000 R CNN
 F 1 "R_2k_0402" H 2900 8100 60  0001 C CNN
-F 2 "antmicro-footprints:0402-res" H 3100 8450 60  0001 L CNN
+F 2 "sc606-baseboard-footprints:0402-res" H 3100 8450 60  0001 L CNN
 F 3 "" H 2900 8250 50  0001 C CNN
 F 4 "VISHAY" H 3100 8650 60  0001 L CNN "Manufacturer"
@@
 $EndComp
 $Comp
-L antmicroResistors0402:R_2k_0402 R?
+L sc606-baseboard:R_2k_0402 R16
 U 1 1 6200206C
 P 2350 8250
-F 0 "R?" V 2500 8250 60  0000 R CNN
+F 0 "R16" V 2500 8250 60  0000 R CNN
 F 1 "R_2k_0402" H 2350 8100 60  0001 C CNN
-F 2 "antmicro-footprints:0402-res" H 2550 8450 60  0001 L CNN
+F 2 "sc606-baseboard-footprints:0402-res" H 2550 8450 60  0001 L CNN
 F 3 "" H 2350 8250 50  0001 C CNN
 F 4 "VISHAY" H 2550 8650 60  0001 L CNN "Manufacturer"
@@
 $EndComp
 $Comp
-L antmicroResistors0402:R_2k_0402 R?
+L sc606-baseboard:R_2k_0402 R17
 U 1 1 62002978
 P 2500 8250
-F 0 "R?" V 2650 8250 60  0000 R CNN
+F 0 "R17" V 2650 8250 60  0000 R CNN
 F 1 "R_2k_0402" H 2500 8100 60  0001 C CNN
-F 2 "antmicro-footprints:0402-res" H 2700 8450 60  0001 L CNN
+F 2 "sc606-baseboard-footprints:0402-res" H 2700 8450 60  0001 L CNN
 F 3 "" H 2500 8250 50  0001 C CNN
 F 4 "VISHAY" H 2700 8650 60  0001 L CNN "Manufacturer"
@@
 CAM_I2C_SCL
 $Comp
-L power:GND #PWR?
+L sc606-baseboard:GND #PWR044
 U 1 1 6206201E
 P 12500 7450
-F 0 "#PWR?" H 12500 7200 50  0001 C CNN
+F 0 "#PWR044" H 12500 7200 50  0001 C CNN
 F 1 "GND" H 12505 7277 50  0000 C CNN
 F 2 "" H 12500 7450 50  0001 C CNN

Commit message: Block diagram update
Parts:
- C33: footprint sc606-baseboard-footprints:0402-cap -> antmicro-footprints:0402-cap; symbol sc606-baseboard:C_100n_0402 -> antmicroCapacitors0402:C_100n_0402
- J3: footprint sc606-baseboard-footprints:WE_68715014522 -> antmicro-footprints:WE_68715014522; symbol sc606-baseboard:WE_68715014522 -> antmicroFCCConnectors:WE_68715014522
- R16, R17, R18, R19, R20, R27, R28, R29, R30: footprint sc606-baseboard-footprints:0402-res -> antmicro-footprints:0402-res; symbol sc606-baseboard:R_2k_0402 -> antmicroResistors0402:R_2k_0402
- R21, R22, R23, R24, R25, R26: footprint sc606-baseboard-footprints:0402-res -> antmicro-footprints:0402-res; symbol sc606-baseboard:R_0R_0402 -> antmicroResistors0402:R_0R_0402
- U3: footprint sc606-baseboard-footprints:TSSOP-8_W3mm -> antmicro-footprints:TSSOP-8_W3mm; symbol sc606-baseboard:NTS0102DP -> antmicroLogicTranslatorsLevelShifters:NTS0102DP
- U4: footprint sc606-baseboard-footprints:VQFN-24 -> antmicro-footprints:VQFN-24; symbol sc606-baseboard:PCA9547BS -> antmicroLogicSignalSwitchesMultiplexersDecoders:PCA9547BS
Changed lines of the file:
@@
 Camera I2C multiplexer\n
 $Comp
-L sc606-baseboard:PCA9547BS U4
+L antmicroLogicSignalSwitchesMultiplexersDecoders:PCA9547BS U4
 U 1 1 61E56C5B
 P 4950 4700
 F 0 "U4" H 4850 6089 60  0000 C CNN
 F 1 "PCA9547BS" H 4850 5983 60  0000 C CNN
-F 2 "sc606-baseboard-footprints:VQFN-24" H 4700 3300 60  0001 C CNN
+F 2 "antmicro-footprints:VQFN-24" H 4700 3300 60  0001 C CNN
 F 3 "https://www.nxp.com/docs/en/data-sheet/PCA9547.pdf" H 4950 4700 60  0001 C CNN
 F 4 " NXP" H 4950 4700 50  0001 C CNN "Manufacturer"
@@
 $EndComp
 $Comp
-L sc606-baseboard:C_100n_0402 C33
+L antmicroCapacitors0402:C_100n_0402 C33
 U 1 1 61E589C6
 P 4000 5100
 F 0 "C33" H 4115 5145 60  0000 L CNN
 F 1 "C_100n_0402" H 4000 4950 60  0001 C CNN
-F 2 "sc606-baseboard-footprints:0402-cap" H 4200 5300 60  0001 L CNN
+F 2 "antmicro-footprints:0402-cap" H 4200 5300 60  0001 L CNN
 F 3 "" H 4000 5100 50  0001 C CNN
 F 4 "Walsin" H 4200 5500 60  0001 L CNN "Manufacturer"
@@
 	4000 3600 4000 4950
 $Comp
-L sc606-baseboard:GND #PWR042
+L power:GND #PWR042
 U 1 1 61E5F2B7
 P 4000 6350
@@
 	3250 3900 2050 3900
 $Comp
-L sc606-baseboard:R_0R_0402 R21
+L antmicroResistors0402:R_0R_0402 R21
 U 1 1 61E63E68
 P 3700 3800
 F 0 "R21" H 3700 4013 60  0000 C CNN
 F 1 "R_0R_0402" H 3700 3650 60  0001 C CNN
-F 2 "sc606-baseboard-footprints:0402-res" H 3900 4000 60  0001 L CNN
+F 2 "antmicro-footprints:0402-res" H 3900 4000 60  0001 L CNN
 F 3 "" H 3700 3800 50  0001 C CNN
 F 4 "PANASONIC" H 3900 4200 60  0001 L CNN "Manufacturer"
@@
 	3850 3800 4450 3800
 $Comp
-L sc606-baseboard:R_0R_0402 R22
+L antmicroResistors0402:R_0R_0402 R22
 U 1 1 61E641DF
 P 3700 3900
 F 0 "R22" H 3700 3777 60  0000 C CNN
 F 1 "R_0R_0402" H 3700 3750 60  0001 C CNN
-F 2 "sc606-baseboard-footprints:0402-res" H 3900 4100 60  0001 L CNN
+F 2 "antmicro-footprints:0402-res" H 3900 4100 60  0001 L CNN
 F 3 "" H 3700 3900 50  0001 C CNN
 F 4 "PANASONIC" H 3900 4300 60  0001 L CNN "Manufacturer"
@@
 	2950 3400 3250 3400
 $Comp
-L sc606-baseboard:R_2k_0402 R19
+L antmicroResistors0402:R_2k_0402 R19
 U 1 1 61E68958
 P 2950 3550
 F 0 "R19" V 2905 3620 60  0000 L CNN
 F 1 "R_2k_0402" H 2950 3400 60  0001 C CNN
-F 2 "sc606-baseboard-footprints:0402-res" H 3150 3750 60  0001 L CNN
+F 2 "antmicro-footprints:0402-res" H 3150 3750 60  0001 L CNN
 F 3 "" H 2950 3550 50  0001 C CNN
 F 4 "VISHAY" H 3150 3950 60  0001 L CNN "Manufacturer"
@@
 $EndComp
 $Comp
-L sc606-baseboard:R_2k_0402 R20
+L antmicroResistors0402:R_2k_0402 R20
 U 1 1 61E68DEE
 P 3250 3550
 F 0 "R20" V 3205 3620 60  0000 L CNN
 F 1 "R_2k_0402" H 3250 3400 60  0001 C CNN
-F 2 "sc606-baseboard-footprints:0402-res" H 3450 3750 60  0001 L CNN
+F 2 "antmicro-footprints:0402-res" H 3450 3750 60  0001 L CNN
 F 3 "" H 3250 3550 50  0001 C CNN
 F 4 "VISHAY" H 3450 3950 60  0001 L CNN "Manufacturer"
@@
 	4450 4500 4450 5800
 $Comp
-L sc606-baseboard:R_0R_0402 R23
+L antmicroResistors0402:R_0R_0402 R23
 U 1 1 61E6A5CA
 P 6150 3600
 F 0 "R23" H 6350 3650 60  0000 C CNN
 F 1 "R_0R_0402" H 6150 3450 60  0001 C CNN
-F 2 "sc606-baseboard-footprints:0402-res" H 6350 3800 60  0001 L CNN
+F 2 "antmicro-footprints:0402-res" H 6350 3800 60  0001 L CNN
 F 3 "" H 6150 3600 50  0001 C CNN
 F 4 "PANASONIC" H 6350 4000 60  0001 L CNN "Manufacturer"
@@
 $EndComp
 $Comp
-L sc606-baseboard:R_0R_0402 R24
+L antmicroResistors0402:R_0R_0402 R24
 U 1 1 61E6AAD1
 P 6150 3700
 F 0 "R24" H 6350 3750 60  0000 C CNN
 F 1 "R_0R_0402" H 6150 3550 60  0001 C CNN
-F 2 "sc606-baseboard-footprints:0402-res" H 6350 3900 60  0001 L CNN
+F 2 "antmicro-footprints:0402-res" H 6350 3900 60  0001 L CNN
 F 3 "" H 6150 3700 50  0001 C CNN
 F 4 "PANASONIC" H 6350 4100 60  0001 L CNN "Manufacturer"
@@
 $EndComp
 $Comp
-L sc606-baseboard:R_0R_0402 R25
+L antmicroResistors0402:R_0R_0402 R25
 U 1 1 61E6AE4A
 P 6150 3900
 F 0 "R25" H 6350 3950 60  0000 C CNN
 F 1 "R_0R_0402" H 6150 3750 60  0001 C CNN
-F 2 "sc606-baseboard-footprints:0402-res" H 6350 4100 60  0001 L CNN
+F 2 "antmicro-footprints:0402-res" H 6350 4100 60  0001 L CNN
 F 3 "" H 6150 3900 50  0001 C CNN
 F 4 "PANASONIC" H 6350 4300 60  0001 L CNN "Manufacturer"
@@
 $EndComp
 $Comp
-L sc606-baseboard:R_0R_0402 R26
+L antmicroResistors0402:R_0R_0402 R26
 U 1 1 61E6B0E9
 P 6150 4000
 F 0 "R26" H 6350 4050 60  0000 C CNN
 F 1 "R_0R_0402" H 6150 3850 60  0001 C CNN
-F 2 "sc606-baseboard-footprints:0402-res" H 6350 4200 60  0001 L CNN
+F 2 "antmicro-footprints:0402-res" H 6350 4200 60  0001 L CNN
 F 3 "" H 6150 4000 50  0001 C CNN
 F 4 "PANASONIC" H 6350 4400 60  0001 L CNN "Manufacturer"
@@
 Camera FFC\n\n
 $Comp
-L sc606-baseboard:WE_68715014522 J3
+L antmicroFCCConnectors:WE_68715014522 J3
 U 1 1 61E964B1
 P 12800 3900
 F 0 "J3" H 12880 3092 50  0000 L CNN
 F 1 "WE_68715014522" H 12880 3001 50  0000 L CNN
-F 2 "sc606-baseboard-footprints:WE_68715014522" H 12600 350 50  0001 C CNN
+F 2 "antmicro-footprints:WE_68715014522" H 12600 350 50  0001 C CNN
 F 3 "https://katalog.we-online.de/em/datasheet/6871xx14522.pdf" H 12800 250 50  0001 C CNN
 F 4 "68715014522 " H 13200 3300 60  0001 L CNN "MPN"
@@
 	12600 6400 10900 6400
 $Comp
-L sc606-baseboard:R_2k_0402 R27
+L antmicroResistors0402:R_2k_0402 R27
 U 1 1 61EAFCF7
 P 10300 5450
 F 0 "R27" H 10250 5350 60  0000 L CNN
 F 1 "R_2k_0402" H 10300 5300 60  0001 C CNN
-F 2 "sc606-baseboard-footprints:0402-res" H 10500 5650 60  0001 L CNN
+F 2 "antmicro-footprints:0402-res" H 10500 5650 60  0001 L CNN
 F 3 "" H 10300 5450 50  0001 C CNN
 F 4 "VISHAY" H 10500 5850 60  0001 L CNN "Manufacturer"
@@
 $EndComp
 $Comp
-L sc606-baseboard:R_2k_0402 R28
+L antmicroResistors0402:R_2k_0402 R28
 U 1 1 61EB041B
 P 10500 5450
 F 0 "R28" H 10450 5350 60  0000 L CNN
 F 1 "R_2k_0402" H 10500 5300 60  0001 C CNN
-F 2 "sc606-baseboard-footprints:0402-res" H 10700 5650 60  0001 L CNN
+F 2 "antmicro-footprints:0402-res" H 10700 5650 60  0001 L CNN
 F 3 "" H 10500 5450 50  0001 C CNN
 F 4 "VISHAY" H 10700 5850 60  0001 L CNN "Manufacturer"
@@
 $EndComp
 $Comp
-L sc606-baseboard:R_2k_0402 R29
+L antmicroResistors0402:R_2k_0402 R29
 U 1 1 61EB08C8
 P 10700 5450
 F 0 "R29" H 10650 5350 60  0000 L CNN
 F 1 "R_2k_0402" H 10700 5300 60  0001 C CNN
-F 2 "sc606-baseboard-footprints:0402-res" H 10900 5650 60  0001 L CNN
+F 2 "antmicro-footprints:0402-res" H 10900 5650 60  0001 L CNN
 F 3 "" H 10700 5450 50  0001 C CNN
 F 4 "VISHAY" H 10900 5850 60  0001 L CNN "Manufacturer"
@@
 $EndComp
 $Comp
-L sc606-baseboard:R_2k_0402 R30
+L antmicroResistors0402:R_2k_0402 R30
 U 1 1 61EB0CC5
 P 10900 5450
 F 0 "R30" H 10850 5350 60  0000 L CNN
 F 1 "R_2k_0402" H 10900 5300 60  0001 C CNN
-F 2 "sc606-baseboard-footprints:0402-res" H 11100 5650 60  0001 L CNN
+F 2 "antmicro-footprints:0402-res" H 11100 5650 60  0001 L CNN
 F 3 "" H 10900 5450 50  0001 C CNN
 F 4 "VISHAY" H 11100 5850 60  0001 L CNN "Manufacturer"
@@
 CAM_I2C_SCL_MUX
 $Comp
-L sc606-baseboard:NTS0102DP U3
+L antmicroLogicTranslatorsLevelShifters:NTS0102DP U3
 U 1 1 61EE57DC
 P 3700 8750
 F 0 "U3" H 3700 9265 50  0000 C CNN
 F 1 "NTS0102DP" H 3700 9174 50  0000 C CNN
-F 2 "sc606-baseboard-footprints:TSSOP-8_W3mm" H 3600 9250 50  0001 C CNN
+F 2 "antmicro-footprints:TSSOP-8_W3mm" H 3600 9250 50  0001 C CNN
 F 3 "" H 4350 9500 50  0001 C CNN
 F 4 "NTS0102DP" H 3650 8350 50  0001 C CNN "MPN"
@@
 $EndComp
 $Comp
-L sc606-baseboard:GND #PWR043
+L power:GND #PWR043
 U 1 1 61EE63E6
 P 4100 9000
@@
 	2900 8800 3300 8800
 $Comp
-L sc606-baseboard:R_2k_0402 R18
+L antmicroResistors0402:R_2k_0402 R18
 U 1 1 61FFF734
 P 2900 8250
 F 0 "R18" V 2950 8450 60  0000 R CNN
 F 1 "R_2k_0402" H 2900 8100 60  0001 C CNN
-F 2 "sc606-baseboard-footprints:0402-res" H 3100 8450 60  0001 L CNN
+F 2 "antmicro-footprints:0402-res" H 3100 8450 60  0001 L CNN
 F 3 "" H 2900 8250 50  0001 C CNN
 F 4 "VISHAY" H 3100 8650 60  0001 L CNN "Manufacturer"
@@
 $EndComp
 $Comp
-L sc606-baseboard:R_2k_0402 R16
+L antmicroResistors0402:R_2k_0402 R16
 U 1 1 6200206C
 P 2350 8250
 F 0 "R16" V 2500 8250 60  0000 R CNN
 F 1 "R_2k_0402" H 2350 8100 60  0001 C CNN
-F 2 "sc606-baseboard-footprints:0402-res" H 2550 8450 60  0001 L CNN
+F 2 "antmicro-footprints:0402-res" H 2550 8450 60  0001 L CNN
 F 3 "" H 2350 8250 50  0001 C CNN
 F 4 "VISHAY" H 2550 8650 60  0001 L CNN "Manufacturer"
@@
 $EndComp
 $Comp
-L sc606-baseboard:R_2k_0402 R17
+L antmicroResistors0402:R_2k_0402 R17
 U 1 1 62002978
 P 2500 8250
 F 0 "R17" V 2650 8250 60  0000 R CNN
 F 1 "R_2k_0402" H 2500 8100 60  0001 C CNN
-F 2 "sc606-baseboard-footprints:0402-res" H 2700 8450 60  0001 L CNN
+F 2 "antmicro-footprints:0402-res" H 2700 8450 60  0001 L CNN
 F 3 "" H 2500 8250 50  0001 C CNN
 F 4 "VISHAY" H 2700 8650 60  0001 L CNN "Manufacturer"
@@
 CAM_I2C_SCL
 $Comp
-L sc606-baseboard:GND #PWR044
+L power:GND #PWR044
 U 1 1 6206201E
 P 12500 7450
