File: peripherals.sch (KiCad schematic (older format))
At the start: 46 parts, among them J1 693022010811, J5 U_FL-R-SMT-1_10_, J6 U_FL-R-SMT-1_10_, J7 DM3AT-SF-PEJM5, U6 NCP163ASN330T1G, U7 EMIF06-MSD02N16

Commit message: Added connectors to LCD displays
Parts:
- removed C55: C_4u7_0402, antmicro-footprints:0402-cap, symbol antmicroCapacitors0402:C_4u7_0402
- removed C56: C_100n_0402, antmicro-footprints:0402-cap, symbol antmicroCapacitors0402:C_100n_0402
- removed D5: PUSB3F96X_PASS, antmicro-footprints:PUSB3F96X, symbol antmicroTVSDiodes:PUSB3F96X_PASS
- removed D6: ESD5Z3_3T1G, antmicro-footprints:SOD-523, symbol antmicroTVSDiodes:ESD5Z3_3T1G
- removed R35, R39: R_2k2_0402, antmicro-footprints:0402-res, symbol antmicroResistors0402:R_2k2_0402
Connections:
- net labels removed: LDO10_2P8, LDO6_1P8, TP0_I2C_SCL, TP0_I2C_SDA, TP0_INT, TP0_RST
- wire segments 150 -> 118
Other:
- note removed: "TP Interface\n\n"
- note removed: "TP connector\n"
Changed lines of the file:
@@
 	2150 1550 2250 1550
 NoConn ~ 2250 1650
-Text Notes 6900 4500 0    98   ~ 20
-TP Interface\n\n
-$Comp
-L antmicroTVSDiodes:PUSB3F96X_PASS D5
-U 1 1 61E35456
-P 7900 6350
-F 0 "D5" H 7900 6000 60  0000 L CNN
-F 1 "PUSB3F96X_PASS" H 7900 5900 60  0000 L CNN
-F 2 "antmicro-footprints:PUSB3F96X" H 8100 5800 60  0001 C CNN
-F 3 "https://pl.mouser.com/datasheet/2/916/PUSB3F96-1600324.pdf" H 7900 6350 60  0001 C CNN
-F 4 "Nexperia" H 8100 5700 50  0001 C CNN "Manufacturer"
-F 5 "PUSB3F96X" H 8100 5700 50  0001 C CNN "MPN"
-	1    7900 6350
-	1    0    0    -1
-$EndComp
-$Comp
-L antmicroTVSDiodes:ESD5Z3_3T1G D6
-U 1 1 61E3EF18
-P 9050 6250
-F 0 "D6" V 9200 6200 60  0000 R CNN
-F 1 "ESD5Z3_3T1G" V 8800 6550 60  0000 R CNN
-F 2 "antmicro-footprints:SOD-523" H 9250 6450 60  0001 L CNN
-F 3 "https://www.onsemi.com/pub/Collateral/ESD5Z2.5T1-D.PDF" H 9250 6550 60  0001 L CNN
-F 4 "ON Semiconductor" H 9250 7350 60  0001 L CNN "Manufacturer"
-F 5 "ESD5Z3.3T1G" H 9250 6750 60  0001 L CNN "MPN"
-	1    9050 6250
-	0    -1   -1   0
-$EndComp
-Text GLabel 7300 5700 0    50   Input ~ 0
-TP0_I2C_SCL
-Text GLabel 7300 5600 0    50   Input ~ 0
-TP0_I2C_SDA
-Text GLabel 7300 5800 0    50   Input ~ 0
-TP0_RST
-Text GLabel 7300 5900 0    50   Input ~ 0
-TP0_INT
-Text GLabel 7300 4950 0    50   Input ~ 0
-LDO6_1P8
-$Comp
-L antmicroResistors0402:R_2k2_0402 R35
-U 1 1 61ED0D15
-P 7500 5250
-F 0 "R35" V 7350 5250 60  0000 L CNN
-F 1 "R_2k2_0402" H 7500 5100 60  0001 C CNN
-F 2 "antmicro-footprints:0402-res" H 7700 5450 60  0001 L CNN
-F 3 "" H 7500 5250 50  0001 C CNN
-F 4 "YAGEO" H 7700 5650 60  0001 L CNN "Manufacturer"
-F 5 "RC0402FR-072K2L" H 7700 5550 60  0001 L CNN "MPN"
-F 6 "2k2" H 7450 5250 50  0000 L CNN "Val"
-	1    7500 5250
-	0    1    1    0
-$EndComp
-$Comp
-L antmicroResistors0402:R_2k2_0402 R39
-U 1 1 61ED1A24
-P 7700 5250
-F 0 "R39" V 7550 5250 60  0000 L CNN
-F 1 "R_2k2_0402" H 7700 5100 60  0001 C CNN
-F 2 "antmicro-footprints:0402-res" H 7900 5450 60  0001 L CNN
-F 3 "" H 7700 5250 50  0001 C CNN
-F 4 "YAGEO" H 7900 5650 60  0001 L CNN "Manufacturer"
-F 5 "RC0402FR-072K2L" H 7900 5550 60  0001 L CNN "MPN"
-F 6 "2k2" H 7650 5250 50  0000 L CNN "Val"
-	1    7700 5250
-	0    1    1    0
-$EndComp
-Wire Wire Line
-	7700 5100 7700 4950
-Wire Wire Line
-	7700 4950 7500 4950
-Wire Wire Line
-	7500 5100 7500 4950
-Connection ~ 7500 4950
-Wire Wire Line
-	7500 4950 7300 4950
-Wire Wire Line
-	7300 5600 7500 5600
-Wire Wire Line
-	7500 5600 7500 5400
-Wire Wire Line
-	7300 5700 7700 5700
-Wire Wire Line
-	7700 5700 7700 5400
-Connection ~ 7500 5600
-Wire Wire Line
-	7700 6150 7700 5700
-Connection ~ 7700 5700
-Wire Wire Line
-	7500 6450 7700 6450
-Wire Wire Line
-	7500 5600 7500 6450
-Wire Wire Line
-	7700 6350 7600 6350
-Wire Wire Line
-	7600 6350 7600 5900
-Wire Wire Line
-	7600 5900 7300 5900
-Wire Wire Line
-	7300 5800 7650 5800
-Wire Wire Line
-	7650 5800 7650 6250
-Wire Wire Line
-	7650 6250 7700 6250
-$Comp
-L power:GND #PWR064
-U 1 1 61F04AE8
-P 7700 6700
-F 0 "#PWR064" H 7700 6450 50  0001 C CNN
-F 1 "GND" H 7705 6527 50  0000 C CNN
-F 2 "" H 7700 6700 50  0001 C CNN
-F 3 "" H 7700 6700 50  0001 C CNN
-	1    7700 6700
-	1    0    0    -1
-$EndComp
-Wire Wire Line
-	7700 6550 7700 6700
-Text GLabel 8750 4950 0    50   Input ~ 0
-LDO10_2P8
-$Comp
-L power:GND #PWR069
-U 1 1 61F2FE2E
-P 9050 6700
-F 0 "#PWR069" H 9050 6450 50  0001 C CNN
-F 1 "GND" H 9055 6527 50  0000 C CNN
-F 2 "" H 9050 6700 50  0001 C CNN
-F 3 "" H 9050 6700 50  0001 C CNN
-	1    9050 6700
-	1    0    0    -1
-$EndComp
-Wire Wire Line
-	9050 6700 9050 6450
-Wire Wire Line
-	9050 6050 9050 4950
-Wire Wire Line
-	9050 4950 8750 4950
-$Comp
-L antmicroCapacitors0402:C_4u7_0402 C55
-U 1 1 61F3D459
-P 9500 6200
-F 0 "C55" H 9500 6300 60  0000 L CNN
-F 1 "C_4u7_0402" H 9500 6050 60  0001 C CNN
-F 2 "antmicro-footprints:0402-cap" H 9700 6400 60  0001 L CNN
-F 3 "" H 9500 6200 50  0001 C CNN
-F 4 "MURATA" H 9700 6600 60  0001 L CNN "Manufacturer"
-F 5 "GRM155R61A475MEAAD" H 9700 6500 60  0001 L CNN "MPN"
-F 6 "4u7" H 9500 6100 50  0000 L CNN "Val"
-	1    9500 6200
-	1    0    0    -1
-$EndComp
-$Comp
-L antmicroCapacitors0402:C_100n_0402 C56
-U 1 1 61F3E80F
-P 9800 6200
-F 0 "C56" H 9800 6300 60  0000 L CNN
-F 1 "C_100n_0402" H 9800 6050 60  0001 C CNN
-F 2 "antmicro-footprints:0402-cap" H 10000 6400 60  0001 L CNN
-F 3 "" H 9800 6200 50  0001 C CNN
-F 4 "Murata" H 10000 6600 60  0001 L CNN "Manufacturer"
-F 5 "GRM155R61H104KE14D" H 10000 6500 60  0001 L CNN "MPN"
-F 6 "100n" H 9800 6100 50  0000 L CNN "Val"
-	1    9800 6200
-	1    0    0    -1
-$EndComp
-$Comp
-L power:GND #PWR071
-U 1 1 61F3F968
-P 9500 6700
-F 0 "#PWR071" H 9500 6450 50  0001 C CNN
-F 1 "GND" H 9505 6527 50  0000 C CNN
-F 2 "" H 9500 6700 50  0001 C CNN
-F 3 "" H 9500 6700 50  0001 C CNN
-	1    9500 6700
-	1    0    0    -1
-$EndComp
-$Comp
-L power:GND #PWR072
-U 1 1 61F3FF72
-P 9800 6700
-F 0 "#PWR072" H 9800 6450 50  0001 C CNN
-F 1 "GND" H 9805 6527 50  0000 C CNN
-F 2 "" H 9800 6700 50  0001 C CNN
-F 3 "" H 9800 6700 50  0001 C CNN
-	1    9800 6700
-	1    0    0    -1
-$EndComp
-Wire Wire Line
-	9800 6700 9800 6350
-Wire Wire Line
-	9500 6350 9500 6700
-Wire Wire Line
-	9800 6050 9500 6050
-Wire Wire Line
-	9050 6050 9500 6050
-Connection ~ 9050 6050
-Connection ~ 9500 6050
-Wire Wire Line
-	7500 5600 10300 5600
-Wire Wire Line
-	7700 5700 10300 5700
-Wire Wire Line
-	7650 5800 10300 5800
-Connection ~ 7650 5800
-Wire Wire Line
-	7600 5900 10300 5900
-Connection ~ 7600 5900
-Wire Wire Line
-	9800 6050 10300 6050
-Connection ~ 9800 6050
-$Comp
-L power:GND #PWR073
-U 1 1 61F8A3E4
-P 10100 6700
-F 0 "#PWR073" H 10100 6450 50  0001 C CNN
-F 1 "GND" H 10105 6527 50  0000 C CNN
-F 2 "" H 10100 6700 50  0001 C CNN
-F 3 "" H 10100 6700 50  0001 C CNN
-	1    10100 6700
-	1    0    0    -1
-$EndComp
-Wire Wire Line
-	10100 6700 10100 6150
-Wire Wire Line
-	10100 6150 10300 6150
 Wire Bus Line
 	700  1450 700  2150
-Text Notes 10450 5900 0    50   ~ 0
-TP connector\n
 $EndSCHEMATC

Commit message: Added keypads and no flag connections to unused pins
Parts:
- added D? (x3): PTVS5V0Z1USKPYL, antmicro-footprints:SOD-964, symbol antmicroTVSDiodes:PTVS5V0Z1USKPYL
- added R? (x3): R_1k_0402, antmicro-footprints:0402-res, symbol antmicroResistors0402:R_1k_0402
- added S? (x3): KMR2, antmicro-footprints:SW_SPST_4.2x2.8, symbol antmicroPushbuttonSwitches:KMR2
- ANT1: footprint antmicro-footprints:GPS-ANT050-mounting-pad -> sc606-baseboard-footprints:GPS-ANT050-mounting-pad; symbol antmicroRFAntennas:GPS-ANT050-external-antenna -> sc606-baseboard:GPS-ANT050-external-antenna
- ANT2: footprint antmicro-footprints:PRO-OB-572_2 -> sc606-baseboard-footprints:PRO-OB-572_2; symbol antmicroRFAntennas:PRO-OB-572_DCPOL -> sc606-baseboard:PRO-OB-572_DCPOL
- C34, C46, C53: footprint antmicro-footprints:0402-cap -> sc606-baseboard-footprints:0402-cap; symbol antmicroCapacitors0402:C_100n_0402 -> sc606-baseboard:C_100n_0402
- C35, C42, C43: footprint antmicro-footprints:0402-cap -> sc606-baseboard-footprints:0402-cap; symbol antmicroCapacitors0402:C_1u_0402 -> sc606-baseboard:C_1u_0402
- C36, C38, C40, C45, C49, C50: footprint antmicro-footprints:0402-cap -> sc606-baseboard-footprints:0402-cap; symbol antmicroCapacitors0402:C_0p5_0402 -> sc606-baseboard:C_0p5_0402
- C37, C41: footprint antmicro-footprints:0402-cap -> sc606-baseboard-footprints:0402-cap; symbol antmicroCapacitors0402:C_0p9_0402 -> sc606-baseboard:C_0p9_0402
- C39: footprint antmicro-footprints:0402-cap -> sc606-baseboard-footprints:0402-cap; symbol antmicroCapacitors0402:C_6p9_0402 -> sc606-baseboard:C_6p9_0402
- C44: footprint antmicro-footprints:0402-cap -> sc606-baseboard-footprints:0402-cap; symbol antmicroCapacitors0402:C_33p_0402 -> sc606-baseboard:C_33p_0402
- C47: footprint antmicro-footprints:0402-cap -> sc606-baseboard-footprints:0402-cap; symbol antmicroCapacitors0402:C_4u7_0402 -> sc606-baseboard:C_4u7_0402
- C48: footprint antmicro-footprints:0402-cap -> sc606-baseboard-footprints:0402-cap; symbol antmicroCapacitors0402:C_100p_0402 -> sc606-baseboard:C_100p_0402
- C51, C52, C54: footprint antmicro-footprints:0402-cap -> sc606-baseboard-footprints:0402-cap; symbol antmicroCapacitors0402:C_22p_0402 -> sc606-baseboard:C_22p_0402
- D2: footprint antmicro-footprints:PUSB3F96X -> sc606-baseboard-footprints:PUSB3F96X; symbol antmicroTVSDiodes:PUSB3F96X_PASS -> sc606-baseboard:PUSB3F96X_PASS
- J1: footprint antmicro-footprints:693022010811 -> sc606-baseboard-footprints:693022010811; symbol antmicroSimCardConnectors:693022010811 -> sc606-baseboard:693022010811
- J5, J6: footprint antmicro-footprints:Coax_Conn_U.FL -> sc606-baseboard-footprints:Coax_Conn_U.FL; symbol antmicroCoaxialConnectorsRF:U_FL-R-SMT-1_10_ -> sc606-baseboard:U_FL-R-SMT-1_10_
- J7: footprint antmicro-footprints:MicroSD_DM3AT-SF-PEJM5 -> sc606-baseboard-footprints:MicroSD_DM3AT-SF-PEJM5; symbol antmicroMemoryConnectorsPCCardSockets:DM3AT-SF-PEJM5 -> sc606-baseboard:DM3AT-SF-PEJM5
- L4: footprint antmicro-footprints:0402-res -> sc606-baseboard-footprints:0402-res; symbol antmicroFixedInductors:LQW15AN2N4B00D -> sc606-baseboard:LQW15AN2N4B00D
- L5: footprint antmicro-footprints:0402-res -> sc606-baseboard-footprints:0402-res; symbol antmicroFixedInductors:MLJ1005HXG56NETD0B -> sc606-baseboard:MLJ1005HXG56NETD0B
- R31, R33: footprint antmicro-footprints:0402-res -> sc606-baseboard-footprints:0402-res; symbol antmicroResistors0402:R_0R_0402 -> sc606-baseboard:R_0R_0402
- R32, R40: footprint antmicro-footprints:0402-res -> sc606-baseboard-footprints:0402-res; symbol antmicroResistors0402:R_10k_0402 -> sc606-baseboard:R_10k_0402
- R34: footprint antmicro-footprints:0603-res -> sc606-baseboard-footprints:0603-res; symbol antmicroResistors0603:R_10R_0603 -> sc606-baseboard:R_10R_0603
- R36, R37, R38: footprint antmicro-footprints:0402-res -> sc606-baseboard-footprints:0402-res; symbol antmicroResistors0402:R_22R_0402 -> sc606-baseboard:R_22R_0402
- U6: footprint antmicro-footprints:SOT-23-5 -> sc606-baseboard-footprints:SOT-23-5; symbol antmicroPMICVoltageRegulatorsLinear:NCP163ASN330T1G -> sc606-baseboard:NCP163ASN330T1G
- U7: footprint antmicro-footprints:UFDFN-16_3.5x1.2mm -> sc606-baseboard-footprints:UFDFN-16_3.5x1.2mm; symbol antmicroPowerProtection:EMIF06-MSD02N16 -> sc606-baseboard:EMIF06-MSD02N16
Connections:
- net labels added: PWRKEY, VOL_DOWN, VOL_UP
- wire segments 118 -> 156
Other:
- note added: "Keypad"

Commit message: Finished connection to HDMI interface. Adjustments after Update of LT9611 symbol
Parts:
- D? (x3): footprint antmicro-footprints:SOD-964 -> sc606-baseboard-footprints:SOD-964; symbol antmicroTVSDiodes:PTVS5V0Z1USKPYL -> sc606-baseboard:PTVS5V0Z1USKPYL
- R? (x3): footprint antmicro-footprints:0402-res -> sc606-baseboard-footprints:0402-res; symbol antmicroResistors0402:R_1k_0402 -> sc606-baseboard:R_1k_0402
- S? (x3): footprint antmicro-footprints:SW_SPST_4.2x2.8 -> sc606-baseboard-footprints:SW_SPST_4.2x2.8; symbol antmicroPushbuttonSwitches:KMR2 -> sc606-baseboard:KMR2
Changed lines of the file:
@@
 PWRKEY
 $Comp
-L antmicroPushbuttonSwitches:KMR2 S?
+L sc606-baseboard:KMR2 S?
 U 1 1 61E2B24F
 P 7950 5150
 F 0 "S?" H 7950 5425 50  0000 C CNN
 F 1 "KMR2" H 7950 5334 50  0000 C CNN
-F 2 "antmicro-footprints:SW_SPST_4.2x2.8" H 8150 5350 50  0001 L CNN
+F 2 "sc606-baseboard-footprints:SW_SPST_4.2x2.8" H 8150 5350 50  0001 L CNN
 F 3 "http://www.farnell.com/datasheets/2631211.pdf" H 8150 5450 60  0001 L CNN
 F 4 "KMR211NGLFS" H 8146 5543 60  0001 L CNN "MPN"
@@
 $EndComp
 $Comp
-L power:GND #PWR0123
+L sc606-baseboard:GND-power #PWR0123
 U 1 1 61E2FDB1
 P 7800 5700
@@
 	7600 5150 7450 5150
 $Comp
-L antmicroResistors0402:R_1k_0402 R?
+L sc606-baseboard:R_1k_0402 R?
 U 1 1 61E46EF8
 P 7250 5150
 F 0 "R?" H 7250 5363 60  0000 C CNN
 F 1 "R_1k_0402" H 7250 5000 60  0001 C CNN
-F 2 "antmicro-footprints:0402-res" H 7450 5350 60  0001 L CNN
+F 2 "sc606-baseboard-footprints:0402-res" H 7450 5350 60  0001 L CNN
 F 3 "" H 7250 5150 50  0001 C CNN
 F 4 "BOURNS" H 7450 5550 60  0001 L CNN "Manufacturer"
@@
 	7100 5150 6950 5150
 $Comp
-L antmicroTVSDiodes:PTVS5V0Z1USKPYL D?
+L sc606-baseboard:PTVS5V0Z1USKPYL D?
 U 1 1 61E533B0
 P 7450 5350
 F 0 "D?" V 7503 5222 60  0000 R CNN
 F 1 "PTVS5V0Z1USKPYL" V 7300 6300 60  0000 R CNN
-F 2 "antmicro-footprints:SOD-964" H 7650 5550 60  0001 L CNN
+F 2 "sc606-baseboard-footprints:SOD-964" H 7650 5550 60  0001 L CNN
 F 3 "https://pl.mouser.com/datasheet/2/916/PTVS5V0Z1USKP-1600477.pdf" H 7650 5650 60  0001 L CNN
 F 4 "Nexperia" H 7650 6450 60  0001 L CNN "Manufacturer"
@@
 VOL_UP
 $Comp
-L antmicroPushbuttonSwitches:KMR2 S?
+L sc606-baseboard:KMR2 S?
 U 1 1 61E6F39D
 P 7950 6550
 F 0 "S?" H 7950 6825 50  0000 C CNN
 F 1 "KMR2" H 7950 6734 50  0000 C CNN
-F 2 "antmicro-footprints:SW_SPST_4.2x2.8" H 8150 6750 50  0001 L CNN
+F 2 "sc606-baseboard-footprints:SW_SPST_4.2x2.8" H 8150 6750 50  0001 L CNN
 F 3 "http://www.farnell.com/datasheets/2631211.pdf" H 8150 6850 60  0001 L CNN
 F 4 "KMR211NGLFS" H 8146 6943 60  0001 L CNN "MPN"
@@
 $EndComp
 $Comp
-L power:GND #PWR0124
+L sc606-baseboard:GND-power #PWR0124
 U 1 1 61E6F3A3
 P 7800 7100
@@
 	7600 6550 7450 6550
 $Comp
-L antmicroResistors0402:R_1k_0402 R?
+L sc606-baseboard:R_1k_0402 R?
 U 1 1 61E6F3B7
 P 7250 6550
 F 0 "R?" H 7250 6763 60  0000 C CNN
 F 1 "R_1k_0402" H 7250 6400 60  0001 C CNN
-F 2 "antmicro-footprints:0402-res" H 7450 6750 60  0001 L CNN
+F 2 "sc606-baseboard-footprints:0402-res" H 7450 6750 60  0001 L CNN
 F 3 "" H 7250 6550 50  0001 C CNN
 F 4 "BOURNS" H 7450 6950 60  0001 L CNN "Manufacturer"
@@
 	7100 6550 6950 6550
 $Comp
-L antmicroTVSDiodes:PTVS5V0Z1USKPYL D?
+L sc606-baseboard:PTVS5V0Z1USKPYL D?
 U 1 1 61E6F3C0
 P 7450 6750
 F 0 "D?" V 7503 6622 60  0000 R CNN
 F 1 "PTVS5V0Z1USKPYL" V 7300 7700 60  0000 R CNN
-F 2 "antmicro-footprints:SOD-964" H 7650 6950 60  0001 L CNN
+F 2 "sc606-baseboard-footprints:SOD-964" H 7650 6950 60  0001 L CNN
 F 3 "https://pl.mouser.com/datasheet/2/916/PTVS5V0Z1USKP-1600477.pdf" H 7650 7050 60  0001 L CNN
 F 4 "Nexperia" H 7650 7850 60  0001 L CNN "Manufacturer"
@@
 VOL_DOWN
 $Comp
-L antmicroPushbuttonSwitches:KMR2 S?
+L sc606-baseboard:KMR2 S?
 U 1 1 61E78403
 P 7950 7800
 F 0 "S?" H 7950 8075 50  0000 C CNN
 F 1 "KMR2" H 7950 7984 50  0000 C CNN
-F 2 "antmicro-footprints:SW_SPST_4.2x2.8" H 8150 8000 50  0001 L CNN
+F 2 "sc606-baseboard-footprints:SW_SPST_4.2x2.8" H 8150 8000 50  0001 L CNN
 F 3 "http://www.farnell.com/datasheets/2631211.pdf" H 8150 8100 60  0001 L CNN
 F 4 "KMR211NGLFS" H 8146 8193 60  0001 L CNN "MPN"
@@
 $EndComp
 $Comp
-L power:GND #PWR0125
+L sc606-baseboard:GND-power #PWR0125
 U 1 1 61E78409
 P 7800 8350
@@
 	7600 7800 7450 7800
 $Comp
-L antmicroResistors0402:R_1k_0402 R?
+L sc606-baseboard:R_1k_0402 R?
 U 1 1 61E7841D
 P 7250 7800
 F 0 "R?" H 7250 8013 60  0000 C CNN
 F 1 "R_1k_0402" H 7250 7650 60  0001 C CNN
-F 2 "antmicro-footprints:0402-res" H 7450 8000 60  0001 L CNN
+F 2 "sc606-baseboard-footprints:0402-res" H 7450 8000 60  0001 L CNN
 F 3 "" H 7250 7800 50  0001 C CNN
 F 4 "BOURNS" H 7450 8200 60  0001 L CNN "Manufacturer"
@@
 	7100 7800 6950 7800
 $Comp
-L antmicroTVSDiodes:PTVS5V0Z1USKPYL D?
+L sc606-baseboard:PTVS5V0Z1USKPYL D?
 U 1 1 61E78426
 P 7450 8000
 F 0 "D?" V 7503 7872 60  0000 R CNN
 F 1 "PTVS5V0Z1USKPYL" V 7300 8950 60  0000 R CNN
-F 2 "antmicro-footprints:SOD-964" H 7650 8200 60  0001 L CNN
+F 2 "sc606-baseboard-footprints:SOD-964" H 7650 8200 60  0001 L CNN
 F 3 "https://pl.mouser.com/datasheet/2/916/PTVS5V0Z1USKP-1600477.pdf" H 7650 8300 60  0001 L CNN
 F 4 "Nexperia" H 7650 9100 60  0001 L CNN "Manufacturer"
