File: power_supply.sch (KiCad schematic (older format))
At the start: 44 parts, among them IC1 TPS54561DPRT, J2 PJ-202A, U1 TPS62823DLCT, U2 TPS62823DLCT

Commit message: Added keypads and no flag connections to unused pins
Parts:
- BAT1: footprint antmicro-footprints:BU1632SM -> sc606-baseboard-footprints:BU1632SM; symbol antmicroBatteryHoldersClipsContacts:BU1632SM -> sc606-baseboard:BU1632SM
- C17, C18, C19: footprint antmicro-footprints:0805-cap -> sc606-baseboard-footprints:0805-cap; symbol antmicroCapacitorsmisc:C_2u2_0805_50V -> sc606-baseboard:C_2u2_0805_50V
- C20: footprint antmicro-footprints:0402-cap -> sc606-baseboard-footprints:0402-cap; symbol antmicroCapacitors0402:C_10n_0402 -> sc606-baseboard:C_10n_0402
- C21: footprint antmicro-footprints:0402-cap -> sc606-baseboard-footprints:0402-cap; symbol antmicroCapacitors0402:C_4n7_0402 -> sc606-baseboard:C_4n7_0402
- C22: footprint antmicro-footprints:0402-cap -> sc606-baseboard-footprints:0402-cap; symbol antmicroCapacitors0402:C_47p_0402 -> sc606-baseboard:C_47p_0402
- C23, C?: footprint antmicro-footprints:0402-cap -> sc606-baseboard-footprints:0402-cap; symbol antmicroCapacitors0402:C_100n_0402 -> sc606-baseboard:C_100n_0402
- C24, C25, C26: footprint antmicro-footprints:0603-cap -> sc606-baseboard-footprints:0603-cap; symbol antmicroCapacitors0603:C_47u_0603 -> sc606-baseboard:C_47u_0603
- C27, C28, C?: footprint antmicro-footprints:0402-cap -> sc606-baseboard-footprints:0402-cap; symbol antmicroCapacitors0402:C_2u2_0402 -> sc606-baseboard:C_2u2_0402
- C29, C30: footprint antmicro-footprints:0603-cap -> sc606-baseboard-footprints:0603-cap; symbol antmicroCapacitors0603:C_100p_0603 -> sc606-baseboard:C_100p_0603
- C31, C32: footprint antmicro-footprints:0402-cap -> sc606-baseboard-footprints:0402-cap; symbol antmicroCapacitors0402:C_10u_0402 -> sc606-baseboard:C_10u_0402
- C?: footprint antmicro-footprints:0402-cap -> sc606-baseboard-footprints:0402-cap; symbol antmicroCapacitors0402:C_1u_0402 -> sc606-baseboard:C_1u_0402
- D3, D4: footprint face-scanner-led-board-footprints:TO-277A -> sc606-baseboard-footprints:TO-277A; symbol antmicroDiodesRectifiersSingle:V8PM45-M3_H -> sc606-baseboard:V8PM45-M3_H
- D?1: footprint antmicro-footprints:PDS760-13 -> sc606-baseboard-footprints:PDS760-13; symbol antmicroDiodesRectifiersSingle:PDS760-13 -> sc606-baseboard:PDS760-13
- IC1: footprint antmicro-footprints:WSON-10_4x4 -> sc606-baseboard-footprints:WSON-10_4x4; symbol antmicroPMICVoltageRegulatorsLinear:TPS54561DPRT -> sc606-baseboard:TPS54561DPRT
- J2: footprint antmicro-footprints:Barrel_Jack_5.5mmODx2.1mmID_PJ-202A -> sc606-baseboard-footprints:Barrel_Jack_5.5mmODx2.1mmID_PJ-202A; symbol antmicroBarrelPowerConnectors:PJ-202A -> sc606-baseboard:PJ-202A
- L1: footprint antmicro-footprints:WE_7447798720 -> sc606-baseboard-footprints:WE_7447798720; symbol antmicroFixedInductors:7447798720 -> sc606-baseboard:7447798720
- L2, L3: footprint antmicro-footprints:IHLP-1212AE -> sc606-baseboard-footprints:IHLP-1212AE; symbol antmicroFixedInductors:IHLP1212AEERR47M11 -> sc606-baseboard:IHLP1212AEERR47M11
- R10, R11, R4: footprint antmicro-footprints:0402-res -> sc606-baseboard-footprints:0402-res; symbol antmicroResistors0402:R_10k_0402 -> sc606-baseboard:R_10k_0402
- R12, R14, R3: footprint antmicro-footprints:0402-res -> sc606-baseboard-footprints:0402-res; symbol antmicroResistors0402:R_243k_0402 -> sc606-baseboard:R_243k_0402
- R13, R15, R8: footprint antmicro-footprints:0402-res -> sc606-baseboard-footprints:0402-res; symbol antmicroResistors0402:R_53k6_0402 -> sc606-baseboard:R_53k6_0402
- R5: footprint antmicro-footprints:0402-res -> sc606-baseboard-footprints:0402-res; symbol antmicroResistors0402:R_16k9_0402 -> sc606-baseboard:R_16k9_0402
- R6: footprint antmicro-footprints:0402-res -> sc606-baseboard-footprints:0402-res; symbol antmicroResistors0402:R_100k_0402 -> sc606-baseboard:R_100k_0402
- R7: footprint antmicro-footprints:0603-res -> sc606-baseboard-footprints:0603-res; symbol antmicroResistors0603:R_49R9_0603 -> sc606-baseboard:R_49R9_0603
- R9: footprint antmicro-footprints:0402-res -> sc606-baseboard-footprints:0402-res; symbol antmicroResistors0402:R_10k2_0402 -> sc606-baseboard:R_10k2_0402
- U1, U2: footprint antmicro-footprints:QFN-8_2x1mm -> sc606-baseboard-footprints:QFN-8_2x1mm; symbol antmicroDCDCConverters:TPS62823DLCT -> sc606-baseboard:TPS62823DLCT
- U?: footprint antmicro-footprints:DFN-4_1.2x1.2mm -> sc606-baseboard-footprints:DFN-4_1.2x1.2mm; symbol antmicroPMICVoltageRegulatorsLinear:LD56050 -> sc606-baseboard:LD56050

Commit message: Change DC/DC converters to match project SA800u
Parts:
- removed C27, C?: C_2u2_0402, sc606-baseboard-footprints:0402-cap, symbol sc606-baseboard:C_2u2_0402
- removed C29, C30: C_100p_0603, sc606-baseboard-footprints:0603-cap, symbol sc606-baseboard:C_100p_0603
- removed C31, C32: C_10u_0402, sc606-baseboard-footprints:0402-cap, symbol sc606-baseboard:C_10u_0402
- removed C?: C_1u_0402, sc606-baseboard-footprints:0402-cap, symbol sc606-baseboard:C_1u_0402
- removed C?: C_100n_0402, sc606-baseboard-footprints:0402-cap, symbol sc606-baseboard:C_100n_0402
- removed L2, L3: IHLP1212AEERR47M11, sc606-baseboard-footprints:IHLP-1212AE, symbol sc606-baseboard:IHLP1212AEERR47M11
- removed R10: R_10k_0402, sc606-baseboard-footprints:0402-res, symbol sc606-baseboard:R_10k_0402
- removed R12, R14: R_243k_0402, sc606-baseboard-footprints:0402-res, symbol sc606-baseboard:R_243k_0402
- removed R13, R15: R_53k6_0402, sc606-baseboard-footprints:0402-res, symbol sc606-baseboard:R_53k6_0402
- removed U1, U2: TPS62823DLCT, sc606-baseboard-footprints:QFN-8_2x1mm, symbol sc606-baseboard:TPS62823DLCT
- removed U?: LD56050, sc606-baseboard-footprints:DFN-4_1.2x1.2mm, symbol sc606-baseboard:LD56050
- added C? (x3): C_100n_0402, antmicro-footprints:0402-cap, symbol antmicroCapacitors0402:C_100n_0402
- added C? (x6): C_22u_0603, antmicro-footprints:0603-cap, symbol antmicroCapacitors0603:C_22u_0603
- added C? (x2): C_2u2_0402, sc606-baseboard-footprints:0402-cap, symbol sc606-baseboard:C_2u2_0402
- added L? (x3): XEL4030-332MEC, antmicro-footprints:Coilcraft-XEL4030, symbol antmicroFixedInductors:XEL4030-332MEC
- added R? (x2): R_31k6_0402, antmicro-footprints:0402-res, symbol antmicroResistors0402:R_31k6_0402
- added R? (x3): R_10k_0402, antmicro-footprints:0402-res, symbol antmicroResistors0402:R_10k_0402
- added R? (x2): R_10k_0402, sc606-baseboard-footprints:0402-res, symbol sc606-baseboard:R_10k_0402
- added R?: R_20k_0402, antmicro-footprints:0402-res, symbol antmicroResistors0402:R_20k_0402
- added U? (x3): AP62301WU-7, antmicro-footprints:TSOT23-6, symbol antmicroDCDCConverters:AP62301WU-7
Connections:
- wire segments 109 -> 135
Other:
- note added: "5V to 1V2 for Lontium9611\n"
- note removed: "5V to 1V2 for Lontium9711\n"
- moved on the sheet: R11

Commit message: Finished connection to HDMI interface. Adjustments after Update of LT9611 symbol
Parts:
- C? (x3): footprint antmicro-footprints:0402-cap -> sc606-baseboard-footprints:0402-cap; symbol antmicroCapacitors0402:C_100n_0402 -> sc606-baseboard:C_100n_0402
- C? (x6): footprint antmicro-footprints:0603-cap -> sc606-baseboard-footprints:0603-cap; symbol antmicroCapacitors0603:C_22u_0603 -> sc606-baseboard:C_22u_0603
- L? (x3): footprint antmicro-footprints:Coilcraft-XEL4030 -> sc606-baseboard-footprints:Coilcraft-XEL4030; symbol antmicroFixedInductors:XEL4030-332MEC -> sc606-baseboard:XEL4030-332MEC
- R? (x2): footprint antmicro-footprints:0402-res -> sc606-baseboard-footprints:0402-res; symbol antmicroResistors0402:R_31k6_0402 -> sc606-baseboard:R_31k6_0402
- R? (x3): footprint antmicro-footprints:0402-res -> sc606-baseboard-footprints:0402-res; symbol antmicroResistors0402:R_10k_0402 -> sc606-baseboard:R_10k_0402
- R?: footprint antmicro-footprints:0402-res -> sc606-baseboard-footprints:0402-res; symbol antmicroResistors0402:R_20k_0402 -> sc606-baseboard:R_20k_0402
- U? (x3): footprint antmicro-footprints:TSOT23-6 -> sc606-baseboard-footprints:TSOT23-6; symbol antmicroDCDCConverters:AP62301WU-7 -> sc606-baseboard:AP62301WU-7
Changed lines of the file:
@@
 1V2_SYS
 $Comp
-L antmicroDCDCConverters:AP62301WU-7 U?
+L sc606-baseboard:AP62301WU-7 U?
 U 1 1 621C43ED
 P 11250 5350
 F 0 "U?" H 11250 5815 50  0000 C CNN
 F 1 "AP62301WU-7" H 11250 5724 50  0000 C CNN
-F 2 "antmicro-footprints:TSOT23-6" H 11200 4700 50  0001 C CNN
+F 2 "sc606-baseboard-footprints:TSOT23-6" H 11200 4700 50  0001 C CNN
 F 3 "https://www.diodes.com/assets/Datasheets/AP62300_AP62301_AP62300T.pdf" H 11200 5000 50  0001 C CNN
 F 4 "AP62301WU-7" H 11200 4800 50  0001 C CNN "MPN"
@@
 $EndComp
 $Comp
-L antmicroCapacitors0402:C_100n_0402 C?
+L sc606-baseboard:C_100n_0402 C?
 U 1 1 621ECBF6
 P 11900 5350
 F 0 "C?" V 11850 5450 60  0000 C CNN
 F 1 "C_100n_0402" H 11900 5200 60  0001 C CNN
-F 2 "antmicro-footprints:0402-cap" H 12100 5550 60  0001 L CNN
+F 2 "sc606-baseboard-footprints:0402-cap" H 12100 5550 60  0001 L CNN
 F 3 "" H 11900 5350 50  0001 C CNN
 F 4 "Murata" H 12100 5750 60  0001 L CNN "Manufacturer"
@@
 	12150 5150 11650 5150
 $Comp
-L antmicroCapacitors0603:C_22u_0603 C?
+L sc606-baseboard:C_22u_0603 C?
 U 1 1 622028CC
 P 13150 5450
 F 0 "C?" H 13150 5550 60  0000 L CNN
 F 1 "C_22u_0603" H 13150 5300 60  0001 C CNN
-F 2 "antmicro-footprints:0603-cap" H 13350 5650 60  0001 L CNN
+F 2 "sc606-baseboard-footprints:0603-cap" H 13350 5650 60  0001 L CNN
 F 3 "" H 13150 5450 50  0001 C CNN
 F 4 "MURATA" H 13350 5850 60  0001 L CNN "Manufacturer"
@@
 $EndComp
 $Comp
-L antmicroCapacitors0603:C_22u_0603 C?
+L sc606-baseboard:C_22u_0603 C?
 U 1 1 62202DBF
 P 13400 5450
 F 0 "C?" H 13400 5550 60  0000 L CNN
 F 1 "C_22u_0603" H 13400 5300 60  0001 C CNN
-F 2 "antmicro-footprints:0603-cap" H 13600 5650 60  0001 L CNN
+F 2 "sc606-baseboard-footprints:0603-cap" H 13600 5650 60  0001 L CNN
 F 3 "" H 13400 5450 50  0001 C CNN
 F 4 "MURATA" H 13600 5850 60  0001 L CNN "Manufacturer"
@@
 	13150 5750 13150 5900
 $Comp
-L antmicroFixedInductors:XEL4030-332MEC L?
+L sc606-baseboard:XEL4030-332MEC L?
 U 1 1 6220F938
 P 12400 5150
 F 0 "L?" H 12400 5451 50  0000 C CNN
 F 1 "XEL4030-332MEC" H 12400 5360 50  0000 C CNN
-F 2 "antmicro-footprints:Coilcraft-XEL4030" H 13200 5400 60  0001 C CNN
+F 2 "sc606-baseboard-footprints:Coilcraft-XEL4030" H 13200 5400 60  0001 C CNN
 F 3 "https://www.coilcraft.com/getmedia/8245f050-f190-4295-8c41-7c03d662ee3d/xel4030.pdf" H 12455 5180 60  0001 C CNN
 F 4 "XEL4030-332MEC" H 12600 5650 50  0001 C CNN "MPN"
@@
 	12550 5150 12750 5150
 $Comp
-L antmicroResistors0402:R_31k6_0402 R?
+L sc606-baseboard:R_31k6_0402 R?
 U 1 1 6222A0AF
 P 12750 5300
 F 0 "R?" V 12705 5370 60  0000 L CNN
 F 1 "R_31k6_0402" H 12750 5150 60  0001 C CNN
-F 2 "antmicro-footprints:0402-res" H 12950 5500 60  0001 L CNN
+F 2 "sc606-baseboard-footprints:0402-res" H 12950 5500 60  0001 L CNN
 F 3 "" H 12750 5300 50  0001 C CNN
 F 4 "Vishay" H 12950 5700 60  0001 L CNN "Manufacturer"
@@
 	12750 5150 13150 5150
 $Comp
-L antmicroResistors0402:R_10k_0402 R?
+L sc606-baseboard:R_10k_0402 R?
 U 1 1 6222B21D
 P 12750 5750
 F 0 "R?" V 12705 5820 60  0000 L CNN
 F 1 "R_10k_0402" H 12750 5600 60  0001 C CNN
-F 2 "antmicro-footprints:0402-res" H 12950 5950 60  0001 L CNN
+F 2 "sc606-baseboard-footprints:0402-res" H 12950 5950 60  0001 L CNN
 F 3 "" H 12750 5750 50  0001 C CNN
 F 4 "VISHAY" H 12950 6150 60  0001 L CNN "Manufacturer"
@@
 	9900 8100 10350 8100
 $Comp
-L antmicroDCDCConverters:AP62301WU-7 U?
+L sc606-baseboard:AP62301WU-7 U?
 U 1 1 62251E9D
 P 11250 8100
 F 0 "U?" H 11250 8565 50  0000 C CNN
 F 1 "AP62301WU-7" H 11250 8474 50  0000 C CNN
-F 2 "antmicro-footprints:TSOT23-6" H 11200 7450 50  0001 C CNN
+F 2 "sc606-baseboard-footprints:TSOT23-6" H 11200 7450 50  0001 C CNN
 F 3 "https://www.diodes.com/assets/Datasheets/AP62300_AP62301_AP62300T.pdf" H 11200 7750 50  0001 C CNN
 F 4 "AP62301WU-7" H 11200 7550 50  0001 C CNN "MPN"
@@
 $EndComp
 $Comp
-L antmicroCapacitors0402:C_100n_0402 C?
+L sc606-baseboard:C_100n_0402 C?
 U 1 1 62251EA6
 P 11900 8100
 F 0 "C?" V 11850 8200 60  0000 C CNN
 F 1 "C_100n_0402" H 11900 7950 60  0001 C CNN
-F 2 "antmicro-footprints:0402-cap" H 12100 8300 60  0001 L CNN
+F 2 "sc606-baseboard-footprints:0402-cap" H 12100 8300 60  0001 L CNN
 F 3 "" H 11900 8100 50  0001 C CNN
 F 4 "Murata" H 12100 8500 60  0001 L CNN "Manufacturer"
@@
 	12150 7900 11650 7900
 $Comp
-L antmicroCapacitors0603:C_22u_0603 C?
+L sc606-baseboard:C_22u_0603 C?
 U 1 1 62251EB4
 P 13150 8200
 F 0 "C?" H 13150 8300 60  0000 L CNN
 F 1 "C_22u_0603" H 13150 8050 60  0001 C CNN
-F 2 "antmicro-footprints:0603-cap" H 13350 8400 60  0001 L CNN
+F 2 "sc606-baseboard-footprints:0603-cap" H 13350 8400 60  0001 L CNN
 F 3 "" H 13150 8200 50  0001 C CNN
 F 4 "MURATA" H 13350 8600 60  0001 L CNN "Manufacturer"
@@
 $EndComp
 $Comp
-L antmicroCapacitors0603:C_22u_0603 C?
+L sc606-baseboard:C_22u_0603 C?
 U 1 1 62251EBD
 P 13400 8200
 F 0 "C?" H 13400 8300 60  0000 L CNN
 F 1 "C_22u_0603" H 13400 8050 60  0001 C CNN
-F 2 "antmicro-footprints:0603-cap" H 13600 8400 60  0001 L CNN
+F 2 "sc606-baseboard-footprints:0603-cap" H 13600 8400 60  0001 L CNN
 F 3 "" H 13400 8200 50  0001 C CNN
 F 4 "MURATA" H 13600 8600 60  0001 L CNN "Manufacturer"
@@
 	13150 8500 13150 8650
 $Comp
-L antmicroFixedInductors:XEL4030-332MEC L?
+L sc606-baseboard:XEL4030-332MEC L?
 U 1 1 62251ECF
 P 12400 7900
 F 0 "L?" H 12400 8201 50  0000 C CNN
 F 1 "XEL4030-332MEC" H 12400 8110 50  0000 C CNN
-F 2 "antmicro-footprints:Coilcraft-XEL4030" H 13200 8150 60  0001 C CNN
+F 2 "sc606-baseboard-footprints:Coilcraft-XEL4030" H 13200 8150 60  0001 C CNN
 F 3 "https://www.coilcraft.com/getmedia/8245f050-f190-4295-8c41-7c03d662ee3d/xel4030.pdf" H 12455 7930 60  0001 C CNN
 F 4 "XEL4030-332MEC" H 12600 8400 50  0001 C CNN "MPN"
@@
 	12550 7900 12750 7900
 $Comp
-L antmicroResistors0402:R_31k6_0402 R?
+L sc606-baseboard:R_31k6_0402 R?
 U 1 1 62251ED9
 P 12750 8050
 F 0 "R?" V 12705 8120 60  0000 L CNN
 F 1 "R_31k6_0402" H 12750 7900 60  0001 C CNN
-F 2 "antmicro-footprints:0402-res" H 12950 8250 60  0001 L CNN
+F 2 "sc606-baseboard-footprints:0402-res" H 12950 8250 60  0001 L CNN
 F 3 "" H 12750 8050 50  0001 C CNN
 F 4 "Vishay" H 12950 8450 60  0001 L CNN "Manufacturer"
@@
 	12750 7900 13150 7900
 $Comp
-L antmicroResistors0402:R_10k_0402 R?
+L sc606-baseboard:R_10k_0402 R?
 U 1 1 62251EE4
 P 12750 8500
 F 0 "R?" V 12705 8570 60  0000 L CNN
 F 1 "R_10k_0402" H 12750 8350 60  0001 C CNN
-F 2 "antmicro-footprints:0402-res" H 12950 8700 60  0001 L CNN
+F 2 "sc606-baseboard-footprints:0402-res" H 12950 8700 60  0001 L CNN
 F 3 "" H 12750 8500 50  0001 C CNN
 F 4 "VISHAY" H 12950 8900 60  0001 L CNN "Manufacturer"
@@
 	1600 9650 2050 9650
 $Comp
-L antmicroDCDCConverters:AP62301WU-7 U?
+L sc606-baseboard:AP62301WU-7 U?
 U 1 1 62287EAD
 P 2950 9650
 F 0 "U?" H 2950 10115 50  0000 C CNN
 F 1 "AP62301WU-7" H 2950 10024 50  0000 C CNN
-F 2 "antmicro-footprints:TSOT23-6" H 2900 9000 50  0001 C CNN
+F 2 "sc606-baseboard-footprints:TSOT23-6" H 2900 9000 50  0001 C CNN
 F 3 "https://www.diodes.com/assets/Datasheets/AP62300_AP62301_AP62300T.pdf" H 2900 9300 50  0001 C CNN
 F 4 "AP62301WU-7" H 2900 9100 50  0001 C CNN "MPN"
@@
 $EndComp
 $Comp
-L antmicroCapacitors0402:C_100n_0402 C?
+L sc606-baseboard:C_100n_0402 C?
 U 1 1 62287EB6
 P 3600 9650
 F 0 "C?" V 3550 9750 60  0000 C CNN
 F 1 "C_100n_0402" H 3600 9500 60  0001 C CNN
-F 2 "antmicro-footprints:0402-cap" H 3800 9850 60  0001 L CNN
+F 2 "sc606-baseboard-footprints:0402-cap" H 3800 9850 60  0001 L CNN
 F 3 "" H 3600 9650 50  0001 C CNN
 F 4 "Murata" H 3800 10050 60  0001 L CNN "Manufacturer"
@@
 	3850 9450 3350 9450
 $Comp
-L antmicroCapacitors0603:C_22u_0603 C?
+L sc606-baseboard:C_22u_0603 C?
 U 1 1 62287EC4
 P 4850 9750
 F 0 "C?" H 4850 9850 60  0000 L CNN
 F 1 "C_22u_0603" H 4850 9600 60  0001 C CNN
-F 2 "antmicro-footprints:0603-cap" H 5050 9950 60  0001 L CNN
+F 2 "sc606-baseboard-footprints:0603-cap" H 5050 9950 60  0001 L CNN
 F 3 "" H 4850 9750 50  0001 C CNN
 F 4 "MURATA" H 5050 10150 60  0001 L CNN "Manufacturer"
@@
 $EndComp
 $Comp
-L antmicroCapacitors0603:C_22u_0603 C?
+L sc606-baseboard:C_22u_0603 C?
 U 1 1 62287ECD
 P 5100 9750
 F 0 "C?" H 5100 9850 60  0000 L CNN
 F 1 "C_22u_0603" H 5100 9600 60  0001 C CNN
-F 2 "antmicro-footprints:0603-cap" H 5300 9950 60  0001 L CNN
+F 2 "sc606-baseboard-footprints:0603-cap" H 5300 9950 60  0001 L CNN
 F 3 "" H 5100 9750 50  0001 C CNN
 F 4 "MURATA" H 5300 10150 60  0001 L CNN "Manufacturer"
@@
 	4450 9850 4450 9750
 $Comp
-L antmicroResistors0402:R_10k_0402 R?
+L sc606-baseboard:R_10k_0402 R?
 U 1 1 622B1791
 P 4450 9600
 F 0 "R?" V 4405 9670 60  0000 L CNN
 F 1 "R_10k_0402" H 4450 9450 60  0001 C CNN
-F 2 "antmicro-footprints:0402-res" H 4650 9800 60  0001 L CNN
+F 2 "sc606-baseboard-footprints:0402-res" H 4650 9800 60  0001 L CNN
 F 3 "" H 4450 9600 50  0001 C CNN
 F 4 "VISHAY" H 4650 10000 60  0001 L CNN "Manufacturer"
@@
 $EndComp
 $Comp
-L antmicroFixedInductors:XEL4030-332MEC L?
+L sc606-baseboard:XEL4030-332MEC L?
 U 1 1 622E2227
 P 4100 9450
 F 0 "L?" H 4100 9751 50  0000 C CNN
 F 1 "XEL4030-332MEC" H 4100 9660 50  0000 C CNN
-F 2 "antmicro-footprints:Coilcraft-XEL4030" H 4900 9700 60  0001 C CNN
+F 2 "sc606-baseboard-footprints:Coilcraft-XEL4030" H 4900 9700 60  0001 C CNN
 F 3 "https://www.coilcraft.com/getmedia/8245f050-f190-4295-8c41-7c03d662ee3d/xel4030.pdf" H 4155 9480 60  0001 C CNN
 F 4 "XEL4030-332MEC" H 4300 9950 50  0001 C CNN "MPN"
@@
 	4450 9450 4850 9450
 $Comp
-L antmicroResistors0402:R_20k_0402 R?
+L sc606-baseboard:R_20k_0402 R?
 U 1 1 622F4B61
 P 4450 10050
 F 0 "R?" V 4405 10120 60  0000 L CNN
 F 1 "R_20k_0402" H 4450 9900 60  0001 C CNN
-F 2 "antmicro-footprints:0402-res" H 4650 10250 60  0001 L CNN
+F 2 "sc606-baseboard-footprints:0402-res" H 4650 10250 60  0001 L CNN
 F 3 "" H 4450 10050 50  0001 C CNN
 F 4 "VISHAY" H 4650 10450 60  0001 L CNN "Manufacturer"
