File: USB.sch (KiCad schematic (older format))
At the start: 15 parts

Commit message: Added USC-C connector and first option of debug UART
Parts:
- added C? (x11): C_100n_0402, antmicro-footprints:0402-cap, symbol antmicroCapacitors0402:C_100n_0402
- added C?: C_4u7_0402, antmicro-footprints:0402-cap, symbol antmicroCapacitors0402:C_4u7_0402
- added C?: C_10u_0402, antmicro-footprints:0402-cap, symbol antmicroCapacitors0402:C_10u_0402
- added C?: C_1u_0402, antmicro-footprints:0402-cap, symbol antmicroCapacitors0402:C_1u_0402
- added D? (x5): PUSB3F96X_PASS, sc606-baseboard-footprints:PUSB3F96X, symbol sc606-baseboard:PUSB3F96X_PASS
- added J?: 1051330001, antmicro-footprints:USB_Micro_B_Female_Vert_1051330001, symbol antmicroUSBDVIHDMIConnectors:1051330001
- added J?: WE_632723300011, antmicro-footprints:WE_632723300011, symbol antmicroUSBDVIHDMIConnectors:WE_632723300011
- added R? (x4): R_0R_0402, antmicro-footprints:0402-res, symbol antmicroResistors0402:R_0R_0402
- added R?: R_4k7_0402, antmicro-footprints:0402-res, symbol antmicroResistors0402:R_4k7_0402
- added R?: R_10k_0402, antmicro-footprints:0402-res, symbol antmicroResistors0402:R_10k_0402
- added SW?: 1X03, antmicro-footprints:MH_1X03_2.54, symbol antmicroRectangularConnectorsHeadersMalePins:1X03
- added TP? (x2): TP_SMD_0_75MM, antmicro-footprints:Testpoint_smd_0_75mm, symbol antmicroTestPoints:TP_SMD_0_75MM
- added U?: CY7C65213A-32LTXI, Package_DFN_QFN:QFN-32-1EP_5x5mm_P0.5mm_EP3.45x3.45mm, symbol Interface_USB:CY7C65213A-32LTXI
- added U?: FT232RQ-REEL, antmicro-footprints:QFN-32-1EP_5x5mm, symbol antmicroInterfaceControllers:FT232RQ-REEL
Connections:
- net GND: now also C?.1, C?.1, C?.1, C?.2, C?.2, C?.2, D?.3 (GND), D?.3 (GND), D?.3 (GND), D?.3 (GND), D?.3 (GND), D?.4 (CH3), D?.5 (CH4), D?.6 (CH4), D?.7 (CH3), D?.8 (GND), D?.8 (GND), D?.8 (GND), D?.8 (GND), D?.8 (GND), J?.5, J?.A1 (GND), J?.A12 (GND), J?.B1 (GND), J?.B12 (GND), J?.SH, J?.Shell (Shield), R?.2, U?.17 (GND), U?.17 (GND), U?.20 (GND), U?.20 (GND), U?.24 (AGND), U?.24 (AGND), U?.26 (TEST), U?.4 (GND), U?.4 (GND)
- net USB_D_N: now also D?.5 (CH4), D?.6 (CH4), J?.A7 (Dn1), J?.B7 (Dn2)
- net USB_D_P: now also D?.4 (CH3), D?.7 (CH3), J?.A6 (Dp1), J?.B6 (Dp2)
- new net: C?.1, C?.1, D?.1 (CH1), D?.10 (CH1), D?.2 (CH2), D?.9 (CH2), J?.1, R?.1, U?.19 (VCC)
- new net: J?.4, TP?.1
- new net: C?.1, J?.A10 (SSRXn2)
- new net: C?.1, J?.A11 (SSRXp2)
- new net: C?.1, J?.A2 (SSTXp1)
- new net: C?.1, J?.A3 (SSTXn1)
- new net: J?.A5 (CC1), R?.2, R?.2
- new net: C?.2, J?.B10 (SSRXn1)
- new net: C?.2, J?.B11 (SSRXp1)
- new net: C?.2, J?.B2 (SSTXp2)
- new net: C?.2, J?.B3 (SSTXn2)
- new net: J?.B5 (CC2), R?.2, R?.2
- new net: J?.B8 (SBU2), TP?.1
- new net: R?.1, R?.2, U?.18 (~RESET)
- new net: C?.2, U?.16 (VCCD)
- new net: C?.2, U?.16 (3V3OUT)
- new net 5V0_SYS: U?.1 (VCCIO)
- new net CC1: R?.1, R?.1
- new net CC2: R?.1, R?.1
- new net DEBUG_UART_RX: D?.1 (CH1), D?.10 (CH1), SW?.1, U?.30 (TXD), U?.30 (TXD)
- new net DEBUG_UART_TX: D?.2 (CH2), D?.9 (CH2), SW?.2, U?.2 (RXD), U?.2 (RXD)
- new net USBC_VBUS: C?.1, C?.2, D?.1 (CH1), D?.10 (CH1), D?.2 (CH2), D?.9 (CH2), J?.A4 (VBUS), J?.A9 (VBUS), J?.B4 (VBUS), J?.B9 (VBUS)
- new net USBSS_RX1_N: C?.2, D?.4 (CH3), D?.7 (CH3)
- new net USBSS_RX1_P: C?.2, D?.5 (CH4), D?.6 (CH4)
- new net USBSS_RX2_N: C?.1, D?.4 (CH3), D?.7 (CH3)
- new net USBSS_RX2_P: C?.1, D?.5 (CH4), D?.6 (CH4)
- new net USBSS_TX1_N: C?.2, D?.2 (CH2), D?.9 (CH2)
- new net USBSS_TX1_P: C?.2, D?.1 (CH1), D?.10 (CH1)
- new net USBSS_TX2_N: C?.1, D?.2 (CH2), D?.9 (CH2)
- new net USBSS_TX2_P: C?.1, D?.1 (CH1), D?.10 (CH1)
- new net USB_DM: D?.5 (CH4), D?.6 (CH4), J?.3, U?.15 (USBDM), U?.15 (USBDM)
- new net USB_DP: D?.4 (CH3), D?.7 (CH3), J?.2, U?.14 (USBDP), U?.14 (USBDP)
- no-connect marks 0 -> 30
Other:
- note added: "3pin goldpin for external dongle to debug using UART.\nMust discuss if 3rd pin will be GND."
- note added: "Debug UART option A"
- note added: "Debug UART option B"
- note added: "USB-C Connector"
- note added: "info: crossed from SoM"

Commit message: Chip changed for Debug UART. Changed connector from USB-A to USB-C
Parts:
- removed C?: C_100n_0402, antmicro-footprints:0402-cap, symbol antmicroCapacitors0402:C_100n_0402
- removed C?: C_4u7_0402, antmicro-footprints:0402-cap, symbol antmicroCapacitors0402:C_4u7_0402
- removed C?: C_1u_0402, antmicro-footprints:0402-cap, symbol antmicroCapacitors0402:C_1u_0402
- removed D? (x3): PUSB3F96X_PASS, sc606-baseboard-footprints:PUSB3F96X, symbol sc606-baseboard:PUSB3F96X_PASS
- removed J?: 1051330001, antmicro-footprints:USB_Micro_B_Female_Vert_1051330001, symbol antmicroUSBDVIHDMIConnectors:1051330001
- removed R?: R_4k7_0402, antmicro-footprints:0402-res, symbol antmicroResistors0402:R_4k7_0402
- removed R?: R_10k_0402, antmicro-footprints:0402-res, symbol antmicroResistors0402:R_10k_0402
- removed TP?: TP_SMD_0_75MM, antmicro-footprints:Testpoint_smd_0_75mm, symbol antmicroTestPoints:TP_SMD_0_75MM
- removed U?: CY7C65213A-32LTXI, Package_DFN_QFN:QFN-32-1EP_5x5mm_P0.5mm_EP3.45x3.45mm, symbol Interface_USB:CY7C65213A-32LTXI
- added C? (x2): C_100n_0402, sc606-baseboard-footprints:0402-cap, symbol sc606-baseboard:C_100n_0402
- added C?: C_2u2_0402, antmicro-footprints:0402-cap, symbol antmicroCapacitors0402:C_2u2_0402
- added C?: C_1u_0402, antmicro-footprints:0402-cap, symbol antmicroCapacitors0402:C_1u_0402
- added C? (x2): C_47p_0402, antmicro-footprints:0402-cap, symbol antmicroCapacitors0402:C_47p_0402
- added D?: 1N4148WS, sc606-baseboard-footprints:SOD-323F, symbol sc606-baseboard:1N4148WS
- added D? (x3): PESD5V0C2BDFZ, sc606-baseboard-footprints:DFN0603-3, symbol sc606-baseboard:PESD5V0C2BDFZ
- added FB?: BLM18EG221SN1D, antmicro-footprints:0603, symbol antmicroFerriteBeadsandChips:BLM18EG221SN1D
- added IC?: TPS7A0518PDBVT, antmicro-footprints:SOT-23-5, symbol antmicroPMICVoltageRegulatorsLinear:TPS7A0518PDBVT
- added J?: WE_632723300011, sc606-baseboard-footprints:WE_632723300011, symbol sc606-baseboard:WE_632723300011
- added U?: USB57442G, antmicro-footprints:QFN40P700X700X100-57N, symbol antmicroInterfaceControllers:USB57442G
- C? (x12): footprint antmicro-footprints:0402-cap -> sc606-baseboard-footprints:0402-cap; symbol antmicroCapacitors0402:C_100n_0402 -> sc606-baseboard:C_100n_0402
- C?: footprint antmicro-footprints:0402-cap -> sc606-baseboard-footprints:0402-cap; symbol antmicroCapacitors0402:C_4u7_0402 -> sc606-baseboard:C_4u7_0402
- C?: footprint antmicro-footprints:0402-cap -> sc606-baseboard-footprints:0402-cap; symbol antmicroCapacitors0402:C_10u_0402 -> sc606-baseboard:C_10u_0402
- J?: footprint antmicro-footprints:USB_Micro_B_Female_Vert_1051330001 -> sc606-baseboard-footprints:USB_Micro_B_Female_Vert_1051330001; symbol antmicroUSBDVIHDMIConnectors:1051330001 -> sc606-baseboard:1051330001
- J?: footprint antmicro-footprints:WE_632723300011 -> sc606-baseboard-footprints:WE_632723300011; symbol antmicroUSBDVIHDMIConnectors:WE_632723300011 -> sc606-baseboard:WE_632723300011
- Q? (x2): footprint antmicro-footprints:SOT-23-3 -> sc606-baseboard-footprints:SOT-23-3; symbol antmicroTransistorsFETsMOSFETsSingle:BSS138-7-F -> sc606-baseboard:BSS138-7-F
- R? (x2): footprint antmicro-footprints:0402-res -> sc606-baseboard-footprints:0402-res; symbol antmicroResistors0402:R_10k_0402 -> sc606-baseboard:R_10k_0402
- R?: footprint antmicro-footprints:0402-res -> sc606-baseboard-footprints:0402-res; symbol antmicroResistors0402:R_1k1_0402 -> sc606-baseboard:R_1k1_0402
- R?: footprint antmicro-footprints:0402-res -> sc606-baseboard-footprints:0402-res; symbol antmicroResistors0402:R_2k2_0402 -> sc606-baseboard:R_2k2_0402
- R? (x5): footprint antmicro-footprints:0402-res -> sc606-baseboard-footprints:0402-res; symbol antmicroResistors0402:R_0R_0402 -> sc606-baseboard:R_0R_0402
- SW?: footprint antmicro-footprints:MH_1X03_2.54 -> sc606-baseboard-footprints:MH_1X03_2.54; symbol antmicroRectangularConnectorsHeadersMalePins:1X03 -> sc606-baseboard:1X03
- TP? (x2): footprint antmicro-footprints:Testpoint_smd_0_75mm -> sc606-baseboard-footprints:Testpoint_smd_0_75mm; symbol antmicroTestPoints:TP_SMD_0_75MM -> sc606-baseboard:TP_SMD_0_75MM
- U?: footprint antmicro-footprints:MSOP-10_W3mm -> sc606-baseboard-footprints:MSOP-10_W3mm; symbol antmicroInterfaceAnalogSwitchesSpecialPurpose:FSUSB30MUX -> sc606-baseboard:FSUSB30MUX
- U?: footprint antmicro-footprints:QFN-32-1EP_5x5mm -> sc606-baseboard-footprints:QFN-32-1EP_5x5mm; symbol antmicroInterfaceControllers:FT232RQ-REEL -> sc606-baseboard:FT232RQ-REEL
Connections:
- net 5V0_SYS: now also D?.A
- net DEBUG_UART_RX: now also D?.1 (CH1)
- net DEBUG_UART_TX: now also D?.2 (CH2)
- net GND: now also SW?.3, U?.33 (EP), C?.2, C?.2, C?.2, C?.2, C?.2, C?.2, D?.3 (GND), D?.3 (GND), D?.3 (GND), IC?.2 (GND), J?.A1 (GND), J?.A12 (GND), J?.B1 (GND), J?.B12 (GND), J?.Shell (Shield), U?.57 (VSS)
- net USBSS_RX1_N: now also C?.1; no longer C?.2
- net USBSS_RX1_P: now also C?.1; no longer C?.2
- net USBSS_RX2_N: now also C?.2; no longer C?.1
- net USBSS_RX2_P: now also C?.2; no longer C?.1
- net USB_D_N: now also D?.2 (CH2); no longer L?.3
- net USB_D_P: now also D?.1 (CH1); no longer L?.2
- net 1V8_DBG: now reaches U?.1 (VCCIO)
- net 1V8_DBG: now also C?.1, C?.1, IC?.5 (VOUT)
- net 5V0_DBG: now reaches U?.19 (VCC)
- net 5V0_DBG: now also C?.1, C?.1, D?.K, FB?.1, IC?.1 (VIN), IC?.3 (EN)
- net USB_DM renamed DBG_USB_D_N
- net DBG_USB_D_N: now also C?.1, D?.2 (CH2), J?.A7 (Dn1), J?.B7 (Dn2)
- net USB_DP renamed DBG_USB_D_P
- net DBG_USB_D_P: now also C?.1, D?.1 (CH1), J?.A6 (Dp1), J?.B6 (Dp2)
- net USB_FLASH_ID renamed SoM_USB_FLASH_ID
- new net: U?.12 (VDD12), U?.15 (VDD12), U?.21 (VDD12), U?.28 (VDD12), U?.33 (VDD12), U?.43 (VDD12), U?.49 (VDD12), U?.5 (VDD12)
- new net: U?.16 (VDD33), U?.31 (VDD33), U?.44 (VDD33), U?.55 (VDD33)
- new net DBG_VBUS: FB?.2, J?.A4 (VBUS), J?.A9 (VBUS), J?.B4 (VBUS), J?.B9 (VBUS)
- new net SoM_USB_D_N: L?.3
- new net SoM_USB_D_P: L?.2
- no-connect marks 30 -> 27
Other:
- note added: "Debug UART"
- note added: "USB HUB"
- note removed: "3pin goldpin for external dongle to debug using UART.\nMust discuss if 3rd pin will be GND."
- note removed: "Debug UART option A"
- note removed: "Debug UART option B"
- moved on the sheet: C?, D?, J?, R?, SW?, TP?, U?

Commit message: Added footprint of 2x USB-A stacked. Added connections to USB HUB.
Parts:
- C?: footprint antmicro-footprints:0402-cap -> sc606-baseboard-footprints:0402-cap; symbol antmicroCapacitors0402:C_2u2_0402 -> sc606-baseboard:C_2u2_0402
- C?: footprint antmicro-footprints:0402-cap -> sc606-baseboard-footprints:0402-cap; symbol antmicroCapacitors0402:C_1u_0402 -> sc606-baseboard:C_1u_0402
- C? (x2): footprint antmicro-footprints:0402-cap -> sc606-baseboard-footprints:0402-cap; symbol antmicroCapacitors0402:C_47p_0402 -> sc606-baseboard:C_47p_0402
- FB?: footprint antmicro-footprints:0603 -> sc606-baseboard-footprints:0603; symbol antmicroFerriteBeadsandChips:BLM18EG221SN1D -> sc606-baseboard:BLM18EG221SN1D
- IC?: footprint antmicro-footprints:SOT-23-5 -> sc606-baseboard-footprints:SOT-23-5; symbol antmicroPMICVoltageRegulatorsLinear:TPS7A0518PDBVT -> sc606-baseboard:TPS7A0518PDBVT
- U?: footprint antmicro-footprints:QFN40P700X700X100-57N -> sc606-baseboard-footprints:QFN40P700X700X100-57N; symbol antmicroInterfaceControllers:USB57442G -> sc606-baseboard:USB57442G
Changed lines of the file:
@@
 5V0_DBG
 $Comp
-L antmicroCapacitors0402:C_2u2_0402 C?
+L sc606-baseboard:C_2u2_0402 C?
 U 1 1 61FA0F2B
 P 4150 6700
 F 0 "C?" H 4265 6745 60  0000 L CNN
 F 1 "C_2u2_0402" H 4150 6550 60  0001 C CNN
-F 2 "antmicro-footprints:0402-cap" H 4350 6900 60  0001 L CNN
+F 2 "sc606-baseboard-footprints:0402-cap" H 4350 6900 60  0001 L CNN
 F 3 "" H 4150 6700 50  0001 C CNN
 F 4 "TDK" H 4350 7100 60  0001 L CNN "Manufacturer"
@@
 $EndComp
 $Comp
-L antmicroCapacitors0402:C_1u_0402 C?
+L sc606-baseboard:C_1u_0402 C?
 U 1 1 61FA1789
 P 5750 6700
 F 0 "C?" H 5865 6745 60  0000 L CNN
 F 1 "C_1u_0402" H 5750 6550 60  0001 C CNN
-F 2 "antmicro-footprints:0402-cap" H 5950 6900 60  0001 L CNN
+F 2 "sc606-baseboard-footprints:0402-cap" H 5950 6900 60  0001 L CNN
 F 3 "" H 5750 6700 50  0001 C CNN
 F 4 "TDK" H 5950 7100 60  0001 L CNN "Manufacturer"
@@
 $EndComp
 $Comp
-L antmicroPMICVoltageRegulatorsLinear:TPS7A0518PDBVT IC?
+L sc606-baseboard:TPS7A0518PDBVT IC?
 U 1 1 61FA2014
 P 5000 6600
 F 0 "IC?" H 5000 7081 50  0000 C CNN
 F 1 "TPS7A0518PDBVT" H 5000 6998 39  0000 C CNN
-F 2 "antmicro-footprints:SOT-23-5" H 5000 6350 50  0001 C CNN
+F 2 "sc606-baseboard-footprints:SOT-23-5" H 5000 6350 50  0001 C CNN
 F 3 "" H 5000 6600 50  0001 C CNN
 F 4 "TPS7A0518PDBVT" H 5000 6915 50  0000 C CNN "MPN"
@@
 	5400 6550 5750 6550
 $Comp
-L power:GND #PWR?
+L sc606-baseboard:GND #PWR?
 U 1 1 61FD04EC
 P 5750 6850
@@
 Connection ~ 5750 6850
 $Comp
-L power:GND #PWR?
+L sc606-baseboard:GND #PWR?
 U 1 1 61FD0C36
 P 4150 6850
@@
 	4450 8400 5250 8400
 $Comp
-L antmicroCapacitors0402:C_47p_0402 C?
+L sc606-baseboard:C_47p_0402 C?
 U 1 1 61FF8CD9
 P 4500 10000
 F 0 "C?" H 4550 10100 60  0000 L CNN
 F 1 "C_47p_0402" H 4500 9850 60  0001 C CNN
-F 2 "antmicro-footprints:0402-cap" H 4700 10200 60  0001 L CNN
+F 2 "sc606-baseboard-footprints:0402-cap" H 4700 10200 60  0001 L CNN
 F 3 "" H 4500 10000 50  0001 C CNN
 F 4 "KEMET" H 4700 10400 60  0001 L CNN "Manufacturer"
@@
 $EndComp
 $Comp
-L antmicroCapacitors0402:C_47p_0402 C?
+L sc606-baseboard:C_47p_0402 C?
 U 1 1 61FF90E8
 P 4250 10000
 F 0 "C?" H 4300 10100 60  0000 L CNN
 F 1 "C_47p_0402" H 4250 9850 60  0001 C CNN
-F 2 "antmicro-footprints:0402-cap" H 4450 10200 60  0001 L CNN
+F 2 "sc606-baseboard-footprints:0402-cap" H 4450 10200 60  0001 L CNN
 F 3 "" H 4250 10000 50  0001 C CNN
 F 4 "KEMET" H 4450 10400 60  0001 L CNN "Manufacturer"
@@
 DBG_VBUS
 $Comp
-L antmicroFerriteBeadsandChips:BLM18EG221SN1D FB?
+L sc606-baseboard:BLM18EG221SN1D FB?
 U 1 1 622B828F
 P 2350 7400
 F 0 "FB?" H 2350 7687 60  0000 C CNN
 F 1 "BLM18EG221SN1D" H 2350 7581 60  0000 C CNN
-F 2 "antmicro-footprints:0603" H 2550 7600 60  0001 L CNN
+F 2 "sc606-baseboard-footprints:0603" H 2550 7600 60  0001 L CNN
 F 3 "" H 2550 7700 60  0001 L CNN
 F 4 "BLM18EG221SN1D" H 2550 7900 60  0001 L CNN "MPN"
@@
 USB_HUB_N
 $Comp
-L antmicroInterfaceControllers:USB57442G U?
+L sc606-baseboard:USB57442G U?
 U 1 1 628E4FAA
 P 11150 3050
 F 0 "U?" H 11150 4720 50  0000 C CNN
 F 1 "USB57442G" H 11150 4629 50  0000 C CNN
-F 2 "antmicro-footprints:QFN40P700X700X100-57N" H 11150 3050 50  0001 C CNN
+F 2 "sc606-baseboard-footprints:QFN40P700X700X100-57N" H 11150 3050 50  0001 C CNN
 F 3 "https://www.snapeda.com/parts/USB5744/2G/Microchip/datasheet/" H 11150 3050 50  0001 C CNN
 F 4 "USB5744" H 11150 4720 50  0001 C CNN "MPN"
@@
 $EndComp
 $Comp
-L power:GND #PWR?
+L sc606-baseboard:GND #PWR?
 U 1 1 62905F3D
 P 12550 4650
