File: USB_HUB_Connectors.sch (KiCad schematic (older format))
At the start: 129 parts, among them IC3 HD3SS3220, IC4 HD3SS3220, J11 USB-A3-C31-D-RA-CS1, J13 USB-A3-C31-D-RA-CS1, U15 USB57442G, Y2 ABM8G-25.000MHZ-B4Y-T

Commit message: Started rearrangement of components. USB connectors changed to 2xUSB-C
Parts:
- removed C138, C142, C143, C144, C145, C153, C154, C155, C156, C157, C159, C160, C161, C162, C163, C164, C165, C166: C_100n_0402, sc606-baseboard-footprints:0402-cap, symbol sc606-baseboard:C_100n_0402
- removed C139, C152: C_10u_0402, sc606-baseboard-footprints:0402-cap, symbol sc606-baseboard:C_10u_0402
- removed C146, C158: C_47u_0603, sc606-baseboard-footprints:0603-cap, symbol sc606-baseboard:C_47u_0603
- removed D25, D26, D29, D30: PUSB3F96X_PASS, sc606-baseboard-footprints:PUSB3F96X, symbol sc606-baseboard:PUSB3F96X_PASS
- removed IC3, IC4: HD3SS3220, sc606-baseboard-footprints:RNH0030A, symbol sc606-baseboard:HD3SS3220
- removed J11, J13: USB-A3-C31-D-RA-CS1, sc606-baseboard-footprints:USB-A3-C31-D-RA-CS1, symbol sc606-baseboard:USB-A3-C31-D-RA-CS1
- removed R130, R142, R144, R160: R_200k_0402, sc606-baseboard-footprints:0402-res, symbol sc606-baseboard:R_200k_0402
- removed R131, R145: R_10k_0402, sc606-baseboard-footprints:0402-res, symbol sc606-baseboard:R_10k_0402
- removed R132, R139, R140, R146, R153, R154: R_2k_0402, sc606-baseboard-footprints:0402-res, symbol sc606-baseboard:R_2k_0402
- removed R138, R143, R147, R148, R149, R150, R151, R152, R161: R_0R_0402, sc606-baseboard-footprints:0402-res, symbol sc606-baseboard:R_0R_0402
- removed R141, R159: R_909k_0402, sc606-baseboard-footprints:0402-res, symbol sc606-baseboard:R_909k_0402
- removed TP20, TP21, TP22, TP25, TP26, TP27: TP_SMD_0_75MM, sc606-baseboard-footprints:Testpoint_smd_0_75mm, symbol sc606-baseboard:TP_SMD_0_75MM
- added C138, C139, C169, C170: C_100u_0805, sc606-baseboard-footprints:0805-cap, symbol sc606-baseboard:C_100u_0805
- added D25, D26: PESD5V0C2BDFZ, sc606-baseboard-footprints:DFN0603-3, symbol sc606-baseboard:PESD5V0C2BDFZ
- added J11, J13: WE_632723300011, sc606-baseboard-footprints:WE_632723300011, symbol sc606-baseboard:WE_632723300011
- added R130, R131, R132: R_0R_0402, sc606-baseboard-footprints:0402-res, symbol sc606-baseboard:R_0R_0402
- R122, R124: DNP DNP -> (none)
- R123: DNP (none) -> DNP
Connections:
- net USB_A1_D_N is gone; now on net USB_C1_D_N: U15.2 (USB2DN_DM1/PRT_DIS_M1)
- net USB_A1_D_P is gone; now on net USB_C1_D_P: U15.1 (USB2DN_DP1/PRT_DIS_P1)
- net USB_A1_SS_RX_N is gone; now on net USB_C1_SS_RX1_N: U15.7 (USB3DN_RXDM1)
- net USB_A1_SS_RX_P is gone; now on net USB_C1_SS_RX1_P: U15.6 (USB3DN_RXDP1)
- net USB_A1_SS_TX_N is gone; now on net USB_C1_SS_TX1_N: U15.4 (USB3DN_TXDM1)
- net USB_A1_SS_TX_P is gone; now on net USB_C1_SS_TX1_P: U15.3 (USB3DN_TXDP1)
- net USB_A2_D_N is gone; now on net USB_C2_D_N: U15.18 (USB2DN_DM3/PRT_DIS_M3)
- net USB_A2_D_P is gone; now on net USB_C2_D_P: U15.17 (USB2DN_DP3/PRT_DIS_P3)
- net USB_A2_SS_RX_N is gone; now on net USB_C2_SS_RX1_N: U15.23 (USB3DN_RXDM3)
- net USB_A2_SS_RX_P is gone; now on net USB_C2_SS_RX1_P: U15.22 (USB3DN_RXDP3)
- net USB_A2_SS_TX_N is gone; now on net USB_C2_SS_TX1_N: U15.20 (USB3DN_TXDM3)
- net USB_A2_SS_TX_P is gone; now on net USB_C2_SS_TX1_P: U15.19 (USB3DN_TXDP3)
- net USB_C1_SS_C_RX_P is gone; now on net USB_C2_SS_C_RX1_P: R137.2
- net USB_C1_SS_C_TX_N is gone; now on net USB_C2_SS_C_RX1_N: R136.2
- net USB_C1_SS_C_TX_P is gone; now on net USB_C2_SS_C_RX2_N: R135.2
- net USB_C1_SS_RX_N is gone; now on net USB_C1_SS_RX2_N: U15.14 (USB3DN_RXDM2)
- net USB_C2_SS_RX_N is gone; now on net USB_C2_SS_RX2_P: U15.30 (USB3DN_RXDM4)
- net USB_C2_SS_RX_P is gone; now on net USB_C2_SS_RX2_N: U15.29 (USB3DN_RXDP4)
- net USB_C2_SS_TX_N is gone; now on net USB_C2_SS_TX2_N: U15.27 (USB3DN_TXDM4)
- net USB_C2_SS_TX_P is gone; now on net USB_C2_SS_TX2_P: U15.26 (USB3DN_TXDP4)
- net 5V0_USB: now also J11.A4 (VBUS), J11.A9 (VBUS), J11.B4 (VBUS), J11.B9 (VBUS), J13.A4 (VBUS), J13.A9 (VBUS), J13.B4 (VBUS), J13.B9 (VBUS); no longer C103.2, C151.2
- net GND: now also C138.1, C139.1, C169.1, C170.1, D25.3 (GND), D26.3 (GND), J11.A12 (GND), J11.Shell (Shield), J13.A12 (GND), J13.Shell (Shield); no longer R133.1, R134.1
- net USB_C1_CC1: now also R131.1; no longer R122.1
- net USB_C1_CC2: now also R132.1; no longer R124.1
- net USB_C1_D_N: now also D25.2 (CH2), J11.A7 (Dn1), J11.B7 (Dn2)
- net USB_C1_D_P: now also D25.1 (CH1), J11.A6 (Dp1), J11.B6 (Dp2)
- net USB_C1_SS_C_TX1_N: now also C102.1, J11.A3 (SSTXn1); no longer C141.1
- net USB_C1_SS_C_TX1_P: now also C94.1, J11.A2 (SSTXp1)
- net USB_C1_SS_C_TX2_N: now also C140.1, J11.B3 (SSTXn2); no longer C102.1
- net USB_C1_SS_C_TX2_P: now also C141.1, J11.B2 (SSTXp2); no longer C94.1
- net USB_C1_SS_RX1_N: now also R130.1
- net USB_C1_SS_RX1_P: now also R133.1
- net USB_C1_SS_RX2_N: now also R124.1; no longer C140.2
- net USB_C1_SS_RX2_P: now also R122.1, U15.13 (USB3DN_RXDP2)
- net USB_C1_SS_TX1_N: now also C102.2; no longer C141.2
- net USB_C1_SS_TX1_P: now also C94.2
- net USB_C1_SS_TX2_N: now also C140.2, U15.11 (USB3DN_TXDM2); no longer C102.2
- net USB_C1_SS_TX2_P: now also C141.2, U15.10 (USB3DN_TXDP2); no longer C94.2
- net USB_C2_CC1: now also R155.1; no longer R158.1
- net USB_C2_CC2: now also R158.1; no longer R155.1
- net USB_C2_D_N: now also D26.2 (CH2), J13.A7 (Dn1), J13.B7 (Dn2)
- net USB_C2_D_P: now also D26.1 (CH1), J13.A6 (Dp1), J13.B6 (Dp2)
- net USB_C2_SS_C_RX1_N: now also J13.B11 (SSRXp1)
- net USB_C2_SS_C_RX1_P: now also J13.B10 (SSRXn1)
- net USB_C2_SS_C_RX2_N: now also J13.A10 (SSRXn2)
- net USB_C2_SS_C_RX2_P: now also R134.2, J13.A11 (SSRXp2)
- net USB_C2_SS_C_TX1_N: now also J13.A3 (SSTXn1)
- net USB_C2_SS_C_TX1_P: now also J13.A2 (SSTXp1)
- net USB_C2_SS_C_TX2_N: now also J13.B3 (SSTXn2)
- net USB_C2_SS_C_TX2_P: now also J13.B2 (SSTXp2)
- net USB_C2_SS_RX1_N: now also R136.1
- net USB_C2_SS_RX1_P: now also R137.1
- net USB_C2_SS_RX2_N: now also D31.5 (CH4), D31.6 (CH4), R135.1; no longer D31.2 (CH2), D31.9 (CH2)
- net USB_C2_SS_RX2_P: now also D31.4 (CH3), D31.7 (CH3), R134.1; no longer D31.1 (CH1), D31.10 (CH1)
- net USB_C2_SS_TX2_N: now also D31.2 (CH2), D31.9 (CH2); no longer D31.5 (CH4), D31.6 (CH4)
- net USB_C2_SS_TX2_P: now also D31.1 (CH1), D31.10 (CH1); no longer D31.4 (CH3), D31.7 (CH3)
- net at R125.2: now also R123.2, J11.A5 (CC1); no longer R124.2
- net at TP18.1: now also J11.A8 (SBU1)
- net USB_C1_SS_C_RX2_P: now reaches R122.2
- net USB_C1_SS_C_RX2_P: now also J11.A11 (SSRXp2); no longer R123.2
- net at TP19.1: now also J11.B8 (SBU2)
- net at R157.2: now also R155.2, J13.B5 (CC2); no longer R158.2
- net at R156.2: now also R158.2, J13.A5 (CC1); no longer R155.2
- net at TP23.1: now also J13.A8 (SBU1)
- net at TP24.1: now also J13.B8 (SBU2)
- net EN1_MUX renamed USB_C1_SS_C_RX1_P
- net USB_C1_SS_C_RX1_P: now also J11.B10 (SSRXn1)
- removed net USB_C1_SS_RX_P: R137.1, U15.13 (USB3DN_RXDP2)
- removed net USB_C1_SS_TX_N: R136.1, U15.11 (USB3DN_TXDM2)
- removed net USB_C1_SS_TX_P: R135.1, U15.10 (USB3DN_TXDP2)
- new net: C151.2, C169.2, C170.2, J13.B1 (GND)
- new net: J11.B5 (CC2), R131.2, R132.2
- new net: C103.2, C138.2, C139.2, J11.B1 (GND)
- new net USB_C1_SS_C_RX1_N: J11.B11 (SSRXp1), R130.2
- new net USB_C1_SS_C_RX2_N: J11.A10 (SSRXn2), R124.2
Other:
- note added: "USB-C connector"
- note removed: "USB-A and USB-C Stack connector"
- moved on the sheet: C133, C135, C147, C148, C149, C150, C151, D28, D31, D32, R121, R155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
