File: serial_and_cameras_interfaces.sch (KiCad schematic (older format))
At the start: 60 parts, among them J13 533980471, J15 533980471, J16 533980471, J17 533980471, J2 WE_68715014522, U16 NTS0102GT, U17 NTS0104PW,118, U18 MAX485EESA, U5 NTS0102GT, U6 PCA9547BS

Commit message: Corrected errors from feedback. Added board name, version, Antmicro and OSHW logo, connector labels, button and LED descriptions
Parts:
- U6: footprint sc606-baseboard-footprints:HVQFN24 -> antmicro-footprints:HVQFN24
Changed lines of the file:
@@
 F 0 "U6" H 8350 4614 60  0000 C CNN
 F 1 "PCA9547BS" H 8350 4508 60  0000 C CNN
-F 2 "sc606-baseboard-footprints:HVQFN24" H 8200 1825 60  0001 C CNN
+F 2 "antmicro-footprints:HVQFN24" H 8200 1825 60  0001 C CNN
 F 3 "https://www.nxp.com/docs/en/data-sheet/PCA9547.pdf" H 8450 3225 60  0001 C CNN
 F 4 " NXP" H 8450 3225 50  0001 C CNN "Manufacturer"

Commit message: Schematic cleanup
Other:
- note added: "Camera and serial interface connectors\n"
- note removed: "Camera connector\n"
- moved on the sheet: C173, R175, R185, R189

Commit message: Corrected footprint of Q10 and Q11. Used 'kmake loclib'
Parts:
- J13, J15, J16, J17: footprint antmicro-footprints:Molex_PicoBlade_53398-0471_1x04-1MP_P1.25mm_Vertical -> sc606-baseboard-footprints:Molex_PicoBlade_53398-0471_1x04-1MP_P1.25mm_Vertical; symbol antmicroRectangularConnectorsHeadersMalePins:533980471 -> sc606-baseboard:533980471
- R186, R187, R188: footprint antmicro-footprints:0402-res -> sc606-baseboard-footprints:0402-res; symbol antmicroResistors0402:R_0R_0402 -> sc606-baseboard:R_0R_0402
- R189: footprint antmicro-footprints:0603-res -> sc606-baseboard-footprints:0603-res; symbol antmicroResistors0603:R_120R_0603 -> sc606-baseboard:R_120R_0603
- U6: footprint antmicro-footprints:HVQFN24 -> sc606-baseboard-footprints:HVQFN24
Changed lines of the file:
@@
 F 0 "U6" H 8350 4614 60  0000 C CNN
 F 1 "PCA9547BS" H 8350 4508 60  0000 C CNN
-F 2 "antmicro-footprints:HVQFN24" H 8200 1825 60  0001 C CNN
+F 2 "sc606-baseboard-footprints:HVQFN24" H 8200 1825 60  0001 C CNN
 F 3 "https://www.nxp.com/docs/en/data-sheet/PCA9547.pdf" H 8450 3225 60  0001 C CNN
 F 4 " NXP" H 8450 3225 50  0001 C CNN "Manufacturer"
@@
 RS485_DIR_GPIO
 $Comp
-L antmicroResistors0402:R_0R_0402 R187
+L sc606-baseboard:R_0R_0402 R187
 U 1 1 621F5421
 P 7100 7775
 F 0 "R187" H 7225 7725 60  0000 L CNN
 F 1 "R_0R_0402" H 7100 7625 60  0001 C CNN
-F 2 "antmicro-footprints:0402-res" H 7300 7975 60  0001 L CNN
+F 2 "sc606-baseboard-footprints:0402-res" H 7300 7975 60  0001 L CNN
 F 3 "" H 7100 7775 50  0001 C CNN
 F 4 "PANASONIC" H 7300 8175 60  0001 L CNN "Manufacturer"
@@
 $EndComp
 $Comp
-L antmicroResistors0402:R_0R_0402 R188
+L sc606-baseboard:R_0R_0402 R188
 U 1 1 6221C459
 P 7100 7875
 F 0 "R188" H 7225 7825 60  0000 L CNN
 F 1 "R_0R_0402" H 7100 7725 60  0001 C CNN
-F 2 "antmicro-footprints:0402-res" H 7300 8075 60  0001 L CNN
+F 2 "sc606-baseboard-footprints:0402-res" H 7300 8075 60  0001 L CNN
 F 3 "" H 7100 7875 50  0001 C CNN
 F 4 "PANASONIC" H 7300 8275 60  0001 L CNN "Manufacturer"
@@
 $EndComp
 $Comp
-L antmicroRectangularConnectorsHeadersMalePins:533980471 J13
+L sc606-baseboard:533980471 J13
 U 1 1 622EC02E
 P 4075 7075
 F 0 "J13" H 3992 6710 50  0000 C CNN
 F 1 "533980471" H 3992 6801 50  0000 C CNN
-F 2 "antmicro-footprints:Molex_PicoBlade_53398-0471_1x04-1MP_P1.25mm_Vertical" H 4175 6975 50  0001 L BNN
+F 2 "sc606-baseboard-footprints:Molex_PicoBlade_53398-0471_1x04-1MP_P1.25mm_Vertical" H 4175 6975 50  0001 L BNN
 F 3 "https://www.molex.com/molex/products/part-detail/pcb_headers/0533980471" H 3975 6875 50  0001 L BNN
 F 4 "Molex" H 4175 7125 50  0001 L BNN "Manufacturer"
@@
 $EndComp
 $Comp
-L antmicroRectangularConnectorsHeadersMalePins:533980471 J15
+L sc606-baseboard:533980471 J15
 U 1 1 62328BC5
 P 4100 8650
 F 0 "J15" H 4017 8285 50  0000 C CNN
 F 1 "533980471" H 4017 8376 50  0000 C CNN
-F 2 "antmicro-footprints:Molex_PicoBlade_53398-0471_1x04-1MP_P1.25mm_Vertical" H 4200 8550 50  0001 L BNN
+F 2 "sc606-baseboard-footprints:Molex_PicoBlade_53398-0471_1x04-1MP_P1.25mm_Vertical" H 4200 8550 50  0001 L BNN
 F 3 "https://www.molex.com/molex/products/part-detail/pcb_headers/0533980471" H 4000 8450 50  0001 L BNN
 F 4 "Molex" H 4200 8700 50  0001 L BNN "Manufacturer"
@@
 $EndComp
 $Comp
-L antmicroRectangularConnectorsHeadersMalePins:533980471 J17
+L sc606-baseboard:533980471 J17
 U 1 1 623298A6
 P 10950 7825
 F 0 "J17" H 10867 7460 50  0000 C CNN
 F 1 "533980471" H 10867 7551 50  0000 C CNN
-F 2 "antmicro-footprints:Molex_PicoBlade_53398-0471_1x04-1MP_P1.25mm_Vertical" H 11050 7725 50  0001 L BNN
+F 2 "sc606-baseboard-footprints:Molex_PicoBlade_53398-0471_1x04-1MP_P1.25mm_Vertical" H 11050 7725 50  0001 L BNN
 F 3 "https://www.molex.com/molex/products/part-detail/pcb_headers/0533980471" H 10850 7625 50  0001 L BNN
 F 4 "Molex" H 11050 7875 50  0001 L BNN "Manufacturer"
@@
 $EndComp
 $Comp
-L antmicroResistors0603:R_120R_0603 R189
+L sc606-baseboard:R_120R_0603 R189
 U 1 1 62401FF8
 P 9925 7825
 F 0 "R189" V 9970 7755 60  0000 R CNN
 F 1 "R_120R_0603" H 9925 7675 60  0001 C CNN
-F 2 "antmicro-footprints:0603-res" H 10125 8025 60  0001 L CNN
+F 2 "sc606-baseboard-footprints:0603-res" H 10125 8025 60  0001 L CNN
 F 3 "" H 9925 7825 50  0001 C CNN
 F 4 "VISHAY" H 10125 8225 60  0001 L CNN "Manufacturer"
@@
 DIR
 $Comp
-L antmicroResistors0402:R_0R_0402 R186
+L sc606-baseboard:R_0R_0402 R186
 U 1 1 6233B85C
 P 7100 7975
 F 0 "R186" H 7225 7925 60  0000 L CNN
 F 1 "R_0R_0402" H 7100 7825 60  0001 C CNN
-F 2 "antmicro-footprints:0402-res" H 7300 8175 60  0001 L CNN
+F 2 "sc606-baseboard-footprints:0402-res" H 7300 8175 60  0001 L CNN
 F 3 "" H 7100 7975 50  0001 C CNN
 F 4 "PANASONIC" H 7300 8375 60  0001 L CNN "Manufacturer"
@@
 	9200 9725 10250 9725
 $Comp
-L antmicroRectangularConnectorsHeadersMalePins:533980471 J16
+L sc606-baseboard:533980471 J16
 U 1 1 623291AA
 P 10925 9775
 F 0 "J16" H 10842 9410 50  0000 C CNN
 F 1 "533980471" H 10842 9501 50  0000 C CNN
-F 2 "antmicro-footprints:Molex_PicoBlade_53398-0471_1x04-1MP_P1.25mm_Vertical" H 11025 9675 50  0001 L BNN
+F 2 "sc606-baseboard-footprints:Molex_PicoBlade_53398-0471_1x04-1MP_P1.25mm_Vertical" H 11025 9675 50  0001 L BNN
 F 3 "https://www.molex.com/molex/products/part-detail/pcb_headers/0533980471" H 10825 9575 50  0001 L BNN
 F 4 "Molex" H 11025 9825 50  0001 L BNN "Manufacturer"
