File: display_module.kicad_sch (KiCad schematic)
At the start: 114 parts, among them J3 F52R-1A7H1-11020, J4 46756-1001, Q3 BSS138APW, Q4 BSS138APW, Q5 BSS138APW, Q6 BSS138APW, U7 LT9611UXC, U8 NTS0102GT, Y1 ABM8G-24.000MHZ-18-D2Y-T

Commit message: Introduce component standardization
Parts:
- C46, C49, C69: footprint sc606-baseboard-footprints:0402-cap -> sc606-baseboard-footprints:C_0402_1005Metric; Author (none) -> Antmicro; License (none) -> Apache-2.0
- C47, C48, C64, C66, C68: footprint sc606-baseboard-footprints:0402-cap -> sc606-baseboard-footprints:C_0402_1005Metric; Author (none) -> Antmicro; License (none) -> Apache-2.0; Manufacturer YAGEO -> Yaego
- C50, C51, C52, C54, C55, C56, C59, C60, C61, C62, C63, C65, C67, C70, C71, C72, C73, C74, C75, C76, C77, C78, C79, C80, C86: footprint sc606-baseboard-footprints:0402-cap -> sc606-baseboard-footprints:C_0402_1005Metric; Author (none) -> Antmicro; Dielectric (none) -> X5R; License (none) -> Apache-2.0; Voltage (none) -> 50V
- C53, C57: footprint sc606-baseboard-footprints:0402-cap -> sc606-baseboard-footprints:C_0402_1005Metric; Author (none) -> Antmicro; License (none) -> Apache-2.0; Manufacturer MULTICOMP -> Multicomp
- C58, C85: footprint sc606-baseboard-footprints:0402-cap -> sc606-baseboard-footprints:C_0402_1005Metric; Author (none) -> Antmicro; License (none) -> Apache-2.0; Manufacturer MURATA -> Murata
- C81, C82: footprint sc606-baseboard-footprints:0402-cap -> sc606-baseboard-footprints:C_0402_1005Metric; Author (none) -> Antmicro; Dielectric (none) -> C0G; License (none) -> Apache-2.0; MPN MC0402N100D500CT -> GCM1555C1H100GA16D; Manufacturer MULTICOMP -> Murata; Voltage (none) -> 50V
- D10: footprint sc606-baseboard-footprints:SOD-323F -> sc606-baseboard-footprints:D_SOD-323F; Author (none) -> Antmicro; License (none) -> Apache-2.0
- D29, D30, D6: footprint sc606-baseboard-footprints:PUSB3F96X -> sc606-baseboard-footprints:Nexperia_DFN-10_2.5x1mm_P0.5mm; Author (none) -> Antmicro; License (none) -> Apache-2.0
- D9: Author (none) -> Antmicro; License (none) -> Apache-2.0
- J3: Author (none) -> Antmicro; License (none) -> Apache-2.0; Manufacturer AMPHENOL ICC -> Amphenol
- J4: value 46756-1001 -> HDMI_Micro-D_46756-1001; symbol sc606-baseboard:46756-1001 -> sc606-baseboard:HDMI_Micro-D_46756-1001; Author (none) -> Antmicro; License (none) -> Apache-2.0
- L10, L11, L12, L16, L17, L18, L19, L8, L9: footprint sc606-baseboard-footprints:FIL_NFP0QHB242HS2D -> sc606-baseboard-footprints:L_Murata_025020_0605Metric; Author (none) -> Antmicro; License (none) -> Apache-2.0; Manufacturer MURATA -> Murata
- L13, L14, L15, L5, L6, L7: value BRC1608TR35M -> L_350n_1.4A_0603; footprint sc606-baseboard-footprints:INDC1608X100N -> sc606-baseboard-footprints:L_0603_1608Metric; symbol sc606-baseboard:BRC1608TR35M -> sc606-baseboard:L_350n_1.4A_0603; Author (none) -> Antmicro; License (none) -> Apache-2.0; Val (none) -> 350n/1.4A
- Q3, Q4, Q5, Q6: value BSS138APW -> BSS138PW; symbol sc606-baseboard:BSS138APW -> sc606-baseboard:BSS138PW; Author (none) -> Antmicro; License (none) -> Apache-2.0; Manufacturer ON Semiconductor -> Nexperia
- R49, R74, R79, R88: footprint sc606-baseboard-footprints:0402-res -> sc606-baseboard-footprints:R_0402_1005Metric; Author (none) -> Antmicro; License (none) -> Apache-2.0; MPN CRCW040210K0FKEDHP -> CR0402-FX-1002GLF; Manufacturer VISHAY -> Bourns; Tolerance (none) -> 1%
- R50, R51, R54, R77, R78: footprint sc606-baseboard-footprints:0402-res -> sc606-baseboard-footprints:R_0402_1005Metric; Author (none) -> Antmicro; License (none) -> Apache-2.0; MPN MCS04020C4701FE000 -> CR0402-FX-4701GLF; Manufacturer VISHAY -> Bourns; Tolerance (none) -> 1%
- R52: value R_1M0_0402 -> R_1M_0402; footprint sc606-baseboard-footprints:0402-res -> sc606-baseboard-footprints:R_0402_1005Metric; symbol sc606-baseboard:R_1M0_0402 -> sc606-baseboard:R_1M_0402; Author (none) -> Antmicro; License (none) -> Apache-2.0; MPN CRG0402F1M0 -> CR0402-FX-1004GLF; Manufacturer TE CONNECTIVITY -> Bourns; Tolerance (none) -> 1%; Val 1M0 -> 1M
- R53: footprint sc606-baseboard-footprints:0402-res -> sc606-baseboard-footprints:R_0402_1005Metric; Author (none) -> Antmicro; License (none) -> Apache-2.0; Manufacturer BOURNS -> Bourns; Tolerance (none) -> 1%
- R55, R56, R61, R62: footprint sc606-baseboard-footprints:0402-res -> sc606-baseboard-footprints:R_0402_1005Metric; Author (none) -> Antmicro; License (none) -> Apache-2.0; MPN RC0402FR-072K2L -> CR0402-FX-2201GLF; Manufacturer YAGEO -> Bourns; Tolerance (none) -> 1%
- R57, R60, R80, R90: footprint sc606-baseboard-footprints:0402-res -> sc606-baseboard-footprints:R_0402_1005Metric; Author (none) -> Antmicro; Current (none) -> 1A; License (none) -> Apache-2.0; Manufacturer PANASONIC -> Panasonic
- R58: footprint sc606-baseboard-footprints:0603-res -> sc606-baseboard-footprints:R_0603_1608Metric; Author (none) -> Antmicro; License (none) -> Apache-2.0; MPN WR06X7681FTL -> CR0603-FX-7681ELF; Manufacturer WALSIN -> Bourns; Tolerance (none) -> 1%
- R59, R89: footprint sc606-baseboard-footprints:0402-res -> sc606-baseboard-footprints:R_0402_1005Metric; Author (none) -> Antmicro; License (none) -> Apache-2.0; MPN CRCW040220K0FKED -> CR0402-FX-2002GLF; Manufacturer VISHAY -> Bourns; Tolerance (none) -> 1%
- R63, R64, R65, R66, R67, R68, R69, R70: footprint sc606-baseboard-footprints:0402-res -> sc606-baseboard-footprints:R_0402_1005Metric; Author (none) -> Antmicro; License (none) -> Apache-2.0; MPN RN73R1ETTP50R0F50 -> CR0402-FX-50R0GLF; Manufacturer KOA -> Bourns; Tolerance (none) -> 1%
- R71, R72, R73: footprint sc606-baseboard-footprints:0402-res -> sc606-baseboard-footprints:R_0402_1005Metric; Author (none) -> Antmicro; License (none) -> Apache-2.0; MPN CRCW04022K00FKED -> CR0402-FX-2001GLF; Manufacturer VISHAY -> Bourns; Tolerance (none) -> 1%
- R75, R76, R81, R82, R84, R85, R86, R87: value R_510_0402 -> R_510R_0402; footprint sc606-baseboard-footprints:0402-res -> sc606-baseboard-footprints:R_0402_1005Metric; symbol sc606-baseboard:R_510_0402 -> sc606-baseboard:R_510R_0402; Author (none) -> Antmicro; License (none) -> Apache-2.0; MPN CRCW0402510RFKEDC -> CR0402-FX-5100GLF; Manufacturer Vishay -> Bourns; Tolerance (none) -> 1%; Val 510 -> 510R
- R83: footprint sc606-baseboard-footprints:0402-res -> sc606-baseboard-footprints:R_0402_1005Metric; Author (none) -> Antmicro; License (none) -> Apache-2.0; MPN ERJ2RKF2702X -> CR0402-FX-2702GLF; Manufacturer PANASONIC_ELECTRONIC_COMPONENTS -> Bourns; Tolerance (none) -> 1%
- TP67, TP68, TP69, TP70: value TP -> TP_1.5mm_SMD; footprint sc606-baseboard-footprints:TP-R-1.5 -> sc606-baseboard-footprints:TP_SMD_1.5mm; symbol sc606-baseboard:TP-antmicroTestPoints -> sc606-baseboard:TP_1.5mm_SMD; Author (none) -> Antmicro; License (none) -> Apache-2.0
- U7: value LT9611UXC -> LT9611; footprint sc606-baseboard-footprints:LT9611 -> sc606-baseboard-footprints:QFN-64-1EP_7.5x7.5mm_P0.4mm; symbol sc606-baseboard:LT9611UXC -> sc606-baseboard:LT9611; Author (none) -> Antmicro; License (none) -> Apache-2.0; Manufacturer LONTIUM -> Lontium
- U8: value NTS0102GT -> NTS0102_XSON; footprint sc606-baseboard-footprints:PSON50P100X195X50-8N -> sc606-baseboard-footprints:XSON-8_1x1.95mm_P0.5mm; symbol sc606-baseboard:NTS0102GT -> sc606-baseboard:NTS0102_XSON; Author (none) -> Antmicro; License (none) -> Apache-2.0; Manufacturer NXP Semiconductors -> NXP
- Y1: footprint sc606-baseboard-footprints:KX-7 -> sc606-baseboard-footprints:Oscillator_SMD_Geyer_KX-7-4Pin_3.2x2.5mm; Author (none) -> Antmicro; License (none) -> Apache-2.0; Manufacturer ABRACON -> Abracon; Val (none) -> 24.000MHz
Connections:
- no-connect marks 19 -> 22
Other:
- note added: "Power flags"
- moved on the sheet: C46, C47, C48, C49, C50, C51, C52, C53, C54, C55, C56, C57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

Commit message: [#61796] Run globlib
Parts:
- C46, C49, C69: footprint sc606-baseboard-footprints:C_0402_1005Metric -> antmicro-footprints:C_0402_1005Metric; symbol sc606-baseboard:C_1u_0402 -> antmicroCapacitors0402:C_1u_0402
- C47, C48, C64, C66, C68: footprint sc606-baseboard-footprints:C_0402_1005Metric -> antmicro-footprints:C_0402_1005Metric; symbol sc606-baseboard:C_10u_0402 -> antmicroCapacitors0402:C_10u_0402
- C50, C51, C52, C54, C55, C56, C59, C60, C61, C62, C63, C65, C67, C70, C71, C72, C73, C74, C75, C76, C77, C78, C79, C80, C86: footprint sc606-baseboard-footprints:C_0402_1005Metric -> antmicro-footprints:C_0402_1005Metric; symbol sc606-baseboard:C_100n_0402 -> antmicroCapacitors0402:C_100n_0402
- C53, C57: footprint sc606-baseboard-footprints:C_0402_1005Metric -> antmicro-footprints:C_0402_1005Metric; symbol sc606-baseboard:C_15p_0402 -> antmicroCapacitors0402:C_15p_0402
- C58, C85: footprint sc606-baseboard-footprints:C_0402_1005Metric -> antmicro-footprints:C_0402_1005Metric; symbol sc606-baseboard:C_4u7_0402 -> antmicroCapacitors0402:C_4u7_0402
- C81, C82: footprint sc606-baseboard-footprints:C_0402_1005Metric -> antmicro-footprints:C_0402_1005Metric; symbol sc606-baseboard:C_10p_0402 -> antmicroCapacitors0402:C_10p_0402
- D10: footprint sc606-baseboard-footprints:D_SOD-323F -> antmicro-footprints:D_SOD-323F; symbol sc606-baseboard:1N4148WS -> antmicroDiodesRectifiersSingle:1N4148WS
- D29, D30, D6: footprint sc606-baseboard-footprints:Nexperia_DFN-10_2.5x1mm_P0.5mm -> antmicro-footprints:Nexperia_DFN-10_2.5x1mm_P0.5mm; symbol sc606-baseboard:PUSB3F96X_PASS -> antmicroTVSDiodes:PUSB3F96X_PASS
- D9: footprint sc606-baseboard-footprints:SOD-123 -> antmicro-footprints:D_SOD-123; symbol sc606-baseboard:1N4148W-7-F -> antmicroDiodesRectifiersSingle:1N4148W-7-F
- J3: footprint sc606-baseboard-footprints:F52R-1A7H1-11020 -> antmicro-footprints:F52R-1A7H1-11020; symbol sc606-baseboard:F52R-1A7H1-11020 -> antmicroFCCConnectors:F52R-1A7H1-11020
- J4: footprint sc606-baseboard-footprints:HDMI_Micro-D_Molex_46765-1x01 -> antmicro-footprints:HDMI-Micro-D_Receptacle_Molex_467651001; symbol sc606-baseboard:HDMI_Micro-D_46756-1001 -> antmicroVideoConnectors:HDMI-Micro-D_Molex_467561001
- L10, L11, L12, L16, L17, L18, L19, L8, L9: footprint sc606-baseboard-footprints:L_Murata_025020_0605Metric -> antmicro-footprints:Choke_025020_0605Metric; symbol sc606-baseboard:NFP0QHB242HS2D -> antmicroCommonModeChokes:Choke_NFP0QHB242HS2D
- L13, L14, L15, L5, L6, L7: footprint sc606-baseboard-footprints:L_0603_1608Metric -> antmicro-footprints:L_0603_1608Metric; symbol sc606-baseboard:L_350n_1.4A_0603 -> antmicroFixedInductors:L_350n_0.81A_0603
- Q3, Q4, Q5, Q6: footprint sc606-baseboard-footprints:SC70-3 -> antmicro-footprints:SC70-3; symbol sc606-baseboard:BSS138PW -> antmicroTransistorsFETsMOSFETsSingle:BSS138PW
- R49, R74, R79, R88: footprint sc606-baseboard-footprints:R_0402_1005Metric -> antmicro-footprints:R_0402_1005Metric; symbol sc606-baseboard:R_10k_0402 -> antmicroResistors0402:R_10k_0402
- R50, R51, R54, R77, R78: footprint sc606-baseboard-footprints:R_0402_1005Metric -> antmicro-footprints:R_0402_1005Metric; symbol sc606-baseboard:R_4k7_0402 -> antmicroResistors0402:R_4k7_0402
- R52: footprint sc606-baseboard-footprints:R_0402_1005Metric -> antmicro-footprints:R_0402_1005Metric; symbol sc606-baseboard:R_1M_0402 -> antmicroResistors0402:R_1M_0402
- R53: footprint sc606-baseboard-footprints:R_0402_1005Metric -> antmicro-footprints:R_0402_1005Metric; symbol sc606-baseboard:R_1k_0402 -> antmicroResistors0402:R_1k_0402
- R55, R56, R61, R62: footprint sc606-baseboard-footprints:R_0402_1005Metric -> antmicro-footprints:R_0402_1005Metric; symbol sc606-baseboard:R_2k2_0402 -> antmicroResistors0402:R_2k2_0402
- R57, R60, R80, R90: footprint sc606-baseboard-footprints:R_0402_1005Metric -> antmicro-footprints:R_0402_1005Metric; symbol sc606-baseboard:R_0R_0402 -> antmicroResistors0402:R_0R_0402
- R58: footprint sc606-baseboard-footprints:R_0603_1608Metric -> antmicro-footprints:R_0603_1608Metric; symbol sc606-baseboard:R_7k68_0603 -> antmicroResistors0603:R_7k68_0603
- R59, R89: footprint sc606-baseboard-footprints:R_0402_1005Metric -> antmicro-footprints:R_0402_1005Metric; symbol sc606-baseboard:R_20k_0402 -> antmicroResistors0402:R_20k_0402
- R63, R64, R65, R66, R67, R68, R69, R70: footprint sc606-baseboard-footprints:R_0402_1005Metric -> antmicro-footprints:R_0402_1005Metric; symbol sc606-baseboard:R_50R_0402 -> antmicroResistors0402:R_50R_0402
- R71, R72, R73: footprint sc606-baseboard-footprints:R_0402_1005Metric -> antmicro-footprints:R_0402_1005Metric; symbol sc606-baseboard:R_2k_0402 -> antmicroResistors0402:R_2k_0402
- R75, R76, R81, R82, R84, R85, R86, R87: footprint sc606-baseboard-footprints:R_0402_1005Metric -> antmicro-footprints:R_0402_1005Metric; symbol sc606-baseboard:R_510R_0402 -> antmicroResistors0402:R_510R_0402
- R83: footprint sc606-baseboard-footprints:R_0402_1005Metric -> antmicro-footprints:R_0402_1005Metric; symbol sc606-baseboard:R_27k_0402 -> antmicroResistors0402:R_27k_0402
- TP67, TP68, TP69, TP70: footprint sc606-baseboard-footprints:TP_SMD_1.5mm -> antmicro-footprints:TP_SMD_1.5mm; symbol sc606-baseboard:TP_1.5mm_SMD -> antmicroTestPoints:TP_1.5mm_SMD
- U7: footprint sc606-baseboard-footprints:QFN-64-1EP_7.5x7.5mm_P0.4mm -> antmicro-footprints:QFN-64-1EP_7.5x7.5mm_P0.4mm; symbol sc606-baseboard:LT9611 -> antmicroInterfaceControllers:LT9611
- U8: footprint sc606-baseboard-footprints:XSON-8_1x1.95mm_P0.5mm -> antmicro-footprints:XSON-8_1x1.95mm_P0.5mm; symbol sc606-baseboard:NTS0102_XSON -> antmicroLogicTranslatorsLevelShifters:NTS0102_XSON
- Y1: footprint sc606-baseboard-footprints:Oscillator_SMD_Geyer_KX-7-4Pin_3.2x2.5mm -> antmicro-footprints:Resonator_SMD_Abracon_ABM8G_3.2x2.5mm; symbol sc606-baseboard:ABM8G-24.000MHZ-18-D2Y-T -> antmicroResonators:Resonator_24MHz_ABM8G

Commit message: [#61796] Update schematics
Parts:
- C47, C64, C66, C68: Manufacturer Yaego -> YAGEO
- C48: Manufacturer Yaego -> YAGEO; now not fitted; now left out of the parts list
- C53, C57: MPN MC0402N150J500CT -> C0402C150K5GACTU.; Manufacturer Multicomp -> KEMET
- C81, C82, R57, R80, R90: now not fitted; now left out of the parts list
- J4: value HDMI_Micro-D_46756-1001 -> HDMI-Micro-D_Molex_467561001
- L10, L11, L12, L16, L17, L18, L19, L8, L9: value NFP0QHB242HS2D -> Choke_NFP0QHB242HS2D; IMax (none) -> 0.1 A
- L13, L14, L15, L5, L6, L7: value L_350n_1.4A_0603 -> L_350n_0.81A_0603; IMax (none) -> 0.81 A; ISat (none) -> 1.4 A; Manufacturer Taiyo Yuden -> TAIYO YUDEN; Size (none) -> 1.6x0.8; Val 350n/1.4A -> 350n/0.81A
- Y1: value ABM8G-24.000MHZ-18-D2Y-T -> Resonator_24MHz_ABM8G; Val 24.000MHz -> 24 MHz
Connections:
- net 5V0_SYS: now also D10.2 (A); no longer D10.A
- net LT9611_VCC33_IO: now also D9.2 (A); no longer D9.A
- net at C85.1, C86.1, J4.19 (+5V)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: now also D10.1 (C); no longer D10.K
- net at R83.1: now also D9.1 (C); no longer D9.K
Other:
- company: (none) -> Antmicro Ltd
- moved on the sheet: R50, R75
