File: power_supply.kicad_sch (KiCad schematic)
At the start: 92 parts, among them IC1 TPS54561QDPRRQ1, Q1 BSS138PW, Q2 BSS138-7-F, U1 AP62301WU-7, U11 AP62301WU-7, U2 AP62301WU-7, U3 AP62301WU-7, U4 74LVC1G123DP,125, U4_1 SN74LVC1G123YZPR

Commit message: [#61796] Run globlib
Parts:
- BAT1: footprint sc606-baseboard-footprints:MS621FE-FL11E -> antmicro-footprints:MS621FE-FL11E; symbol sc606-baseboard:Battery_Holder_MS621FE-FL11E -> antmicroBatteryHoldersClipsContacts:Battery_Holder_MS621FE-FL11E
- C17, C18, C19: footprint sc606-baseboard-footprints:C_0805_2012Metric -> antmicro-footprints:C_0805_2012Metric; symbol sc606-baseboard:C_2u2_0805_50V -> antmicroCapacitorsmisc:C_2u2_0805_50V
- C175, C21, C31, C32, C33, C37, C38: footprint sc606-baseboard-footprints:C_0402_1005Metric -> antmicro-footprints:C_0402_1005Metric; symbol sc606-baseboard:C_10u_0402 -> antmicroCapacitors0402:C_10u_0402
- C176, C24, C25, C34, C35, C36: footprint sc606-baseboard-footprints:C_0402_1005Metric -> antmicro-footprints:C_0402_1005Metric; symbol sc606-baseboard:C_100n_0402 -> antmicroCapacitors0402:C_100n_0402
- C177, C178: footprint sc606-baseboard-footprints:C_0402_1005Metric -> antmicro-footprints:C_0402_1005Metric; symbol sc606-baseboard:C_22u_0402 -> antmicroCapacitors0402:C_22u_0402
- C20: footprint sc606-baseboard-footprints:C_0402_1005Metric -> antmicro-footprints:C_0402_1005Metric; symbol sc606-baseboard:C_10n_0402 -> antmicroCapacitors0402:C_10n_0402
- C22: footprint sc606-baseboard-footprints:C_0402_1005Metric -> antmicro-footprints:C_0402_1005Metric; symbol sc606-baseboard:C_4n7_0402 -> antmicroCapacitors0402:C_4n7_0402
- C23: footprint sc606-baseboard-footprints:C_0402_1005Metric -> antmicro-footprints:C_0402_1005Metric; symbol sc606-baseboard:C_47p_0402 -> antmicroCapacitors0402:C_47p_0402
- C26, C27, C39, C40, C41, C42: footprint sc606-baseboard-footprints:C_0603_1608Metric -> antmicro-footprints:C_0603_1608Metric; symbol sc606-baseboard:C_22u_0603 -> antmicroCapacitors0603:C_22u_0603
- C28, C29, C30: footprint sc606-baseboard-footprints:C_0603_1608Metric -> antmicro-footprints:C_0603_1608Metric; symbol sc606-baseboard:C_47u_0603 -> antmicroCapacitors0603:C_47u_0603
- D2: footprint sc606-baseboard-footprints:PowerDI5 -> antmicro-footprints:PowerDI5; symbol sc606-baseboard:PDS760 -> antmicroDiodesRectifiersSingle:PDS760
- IC1: footprint sc606-baseboard-footprints:WSON-10-1EP_4x4mm_P0.8mm_EP2.6x3mm -> antmicro-footprints:WSON-10-1EP_4x4mm_P0.8mm_EP2.6x3mm; symbol sc606-baseboard:TPS54561QDPRRQ1 -> antmicroPMICVoltageRegulatorsLinear:TPS54561QDPRRQ1
- L1, L23, L3, L4: footprint sc606-baseboard-footprints:L_Coilcraft_XEL4030 -> antmicro-footprints:L_Coilcraft-XEL4030; symbol sc606-baseboard:L_3u3_5.9A_XEL4030 -> antmicroFixedInductors:L_3u3_6.6A_XEL4030
- L2: footprint sc606-baseboard-footprints:L_WE-PDF -> antmicro-footprints:L_WE-PDF-1064; symbol sc606-baseboard:L_7u2_7.9A_WE-PDF -> antmicroFixedInductors:L_7u2_7.9A_WE-PDF-1064
- Q1: footprint sc606-baseboard-footprints:SC70-3 -> antmicro-footprints:SC70-3; symbol sc606-baseboard:BSS138PW -> antmicroTransistorsFETsMOSFETsSingle:BSS138PW
- Q2: footprint sc606-baseboard-footprints:SOT-23-3 -> antmicro-footprints:SOT-23-3; symbol sc606-baseboard:BSS138-7-F -> antmicroTransistorsFETsMOSFETsSingle:BSS138-7-F
- R10, R211, R29, R31: footprint sc606-baseboard-footprints:R_0402_1005Metric -> antmicro-footprints:R_0402_1005Metric; symbol sc606-baseboard:R_10k_0402 -> antmicroResistors0402:R_10k_0402
- R11: footprint sc606-baseboard-footprints:R_0402_1005Metric -> antmicro-footprints:R_0402_1005Metric; symbol sc606-baseboard:R_20k_0402 -> antmicroResistors0402:R_20k_0402
- R12, R17, R19, R207, R22, R27, R7: footprint sc606-baseboard-footprints:R_0402_1005Metric -> antmicro-footprints:R_0402_1005Metric; symbol sc606-baseboard:R_100k_0402 -> antmicroResistors0402:R_100k_0402
- R13: footprint sc606-baseboard-footprints:R_0603_1608Metric -> antmicro-footprints:R_0603_1608Metric; symbol sc606-baseboard:R_49R9_0603 -> antmicroResistors0603:R_49R9_0603
- R14: footprint sc606-baseboard-footprints:R_0402_1005Metric -> antmicro-footprints:R_0402_1005Metric; symbol sc606-baseboard:R_53k6_0402 -> antmicroResistors0402:R_53k6_0402
- R15: footprint sc606-baseboard-footprints:R_0402_1005Metric -> antmicro-footprints:R_0402_1005Metric; symbol sc606-baseboard:R_10k2_0402 -> antmicroResistors0402:R_10k2_0402
- R16, R25: footprint sc606-baseboard-footprints:R_0402_1005Metric -> antmicro-footprints:R_0402_1005Metric; symbol sc606-baseboard:R_100R_0402 -> antmicroResistors0402:R_100R_0402
- R18, R20, R208, R21, R23, R24, R8: footprint sc606-baseboard-footprints:R_0402_1005Metric -> antmicro-footprints:R_0402_1005Metric; symbol sc606-baseboard:R_0R_0402 -> antmicroResistors0402:R_0R_0402
- R209, R5: footprint sc606-baseboard-footprints:R_0402_1005Metric -> antmicro-footprints:R_0402_1005Metric; symbol sc606-baseboard:R_18k_0402 -> antmicroResistors0402:R_18k_0402
- R210: footprint sc606-baseboard-footprints:R_0402_1005Metric -> antmicro-footprints:R_0402_1005Metric; symbol sc606-baseboard:R_22k_0402 -> antmicroResistors0402:R_22k_0402
- R212, R213, R214, R215, R216: footprint sc606-baseboard-footprints:R_1206_3216Metric -> antmicro-footprints:R_1206_3216Metric; symbol sc606-baseboard:R_0R_1206 -> antmicroResistorsmisc:R_0R_1206
- R26: footprint sc606-baseboard-footprints:R_0402_1005Metric -> antmicro-footprints:R_0402_1005Metric; symbol sc606-baseboard:R_180k_0402 -> antmicroResistors0402:R_180k_0402
- R28, R30: footprint sc606-baseboard-footprints:R_0402_1005Metric -> antmicro-footprints:R_0402_1005Metric; symbol sc606-baseboard:R_31k6_0402 -> antmicroResistors0402:R_31k6_0402
- R32: footprint sc606-baseboard-footprints:R_0402_1005Metric -> antmicro-footprints:R_0402_1005Metric; symbol sc606-baseboard:R_1k_0402 -> antmicroResistors0402:R_1k_0402
- R4: footprint sc606-baseboard-footprints:R_0402_1005Metric -> antmicro-footprints:R_0402_1005Metric; symbol sc606-baseboard:R_120k_0402 -> antmicroResistors0402:R_120k_0402
- R6: footprint sc606-baseboard-footprints:R_0402_1005Metric -> antmicro-footprints:R_0402_1005Metric; symbol sc606-baseboard:R_243k_0402 -> antmicroResistors0402:R_243k_0402
- R9: footprint sc606-baseboard-footprints:R_0402_1005Metric -> antmicro-footprints:R_0402_1005Metric; symbol sc606-baseboard:R_16k9_0402 -> antmicroResistors0402:R_16k9_0402
- TP3, TP55, TP56, TP57, TP58, TP59, TP60: footprint sc606-baseboard-footprints:TP_SMD_1.5mm -> antmicro-footprints:TP_SMD_1.5mm; symbol sc606-baseboard:TP_1.5mm_SMD -> antmicroTestPoints:TP_1.5mm_SMD
- U1, U11, U2, U3: footprint sc606-baseboard-footprints:AP62301WU-7-TSOT23-6 -> antmicro-footprints:TSOT23-6; symbol sc606-baseboard:AP62301WU-7 -> antmicroDCDCConverters:AP62301_TSOT
- U4: footprint sc606-baseboard-footprints:TSSOP-8_3x3mm_P0.65mm -> antmicro-footprints:TSSOP-8_3x3mm_P0.65mm; symbol sc606-baseboard:74LVC1G123DP,125 -> antmicroLogicBuffersDriversReceiversTransceivers:74LVC1G123DP,125
- U4_1: footprint sc606-baseboard-footprints:Texas_DSBGA-8_1.9x0.9mm_2x4_P0.5mm -> antmicro-footprints:Texas_DSBGA-8_1.9x0.9mm_Layout2x4_P0.5mm; symbol sc606-baseboard:SN74LVC1G123YZPR -> antmicroLogicBuffersDriversReceiversTransceivers:SN74LVC1G123YZPR

Commit message: [#61796] Update schematics
Parts:
- BAT1: Manufacturer Seiko -> Seiko Instruments
- C17, C18, C19: Val 2u2 50V -> 2u2
- C175, C21, C31, C32, C33, C37, C38: Manufacturer Yaego -> YAGEO
- C177, C178: MPN 04024W226MAT2A -> GRM158R60J226ME01D; Manufacturer AVX -> Murata
- C23: MPN GRM1555C1E470JA01D -> C0402C470J5GACTU; Manufacturer Murata -> KEMET
- L1, L23, L3, L4: value L_3u3_5.9A_XEL4030 -> L_3u3_6.6A_XEL4030; IMax (none) -> 6.6 A; ISat (none) -> 5.9 A; Size 4x4 -> 4.0x4.0; Val 3u3/5.9A -> 3u3/6.6A
- L2: value L_7u2_7.9A_WE-PDF -> L_7u2_7.9A_WE-PDF-1064; IMax (none) -> 7.9 A; ISat (none) -> 6 A
- R18, R20, R208, R8, U4_1: now not fitted; now left out of the parts list
- R212, R213, R214, R215, R216: Manufacturer Multicomp -> Multicomp Pro
- U1, U11, U2, U3: value AP62301WU-7 -> AP62301_TSOT
Connections:
- net GND: now also D2.2 (A); no longer D2.A
- net at C25.2, IC1.9 (SW), L2.1: now also D2.1 (C); no longer D2.C
Other:
- company: (none) -> Antmicro Ltd
- moved on the sheet: R207, R4
