File: USB_flash_debug.kicad_sch (KiCad schematic)
At the start: 30 parts, among them IC2 TPS7A0518PDBVT, J6 E8124-015-01, J9 E8124-015-01, Q7 BSS138-7-F, SW1 1X03, U13 FT232RQ-REEL, U9 FSUSB30MUX

Commit message: Introduce component standardization
Parts:
- C108, C109, C113, C116, C117, C142: footprint sc606-baseboard-footprints:0402-cap -> sc606-baseboard-footprints:C_0402_1005Metric; Author (none) -> Antmicro; Dielectric (none) -> X5R; License (none) -> Apache-2.0; Voltage (none) -> 50V
- C110, C143: footprint sc606-baseboard-footprints:0402-cap -> sc606-baseboard-footprints:C_0402_1005Metric; Author (none) -> Antmicro; License (none) -> Apache-2.0; Manufacturer MURATA -> Murata
- C111, C115: footprint sc606-baseboard-footprints:0402-cap -> sc606-baseboard-footprints:C_0402_1005Metric; Author (none) -> Antmicro; License (none) -> Apache-2.0
- C112, C114: footprint sc606-baseboard-footprints:0402-cap -> sc606-baseboard-footprints:C_0402_1005Metric; Author (none) -> Antmicro; Dielectric (none) -> C0G; License (none) -> Apache-2.0; MPN C0402C470J5GACTU -> GRM1555C1E470JA01D; Manufacturer KEMET -> Murata
- D20, D21, D23: footprint sc606-baseboard-footprints:PUSB3F96X -> sc606-baseboard-footprints:Nexperia_DFN-10_2.5x1mm_P0.5mm; Author (none) -> Antmicro; License (none) -> Apache-2.0
- D22, D43: footprint sc606-baseboard-footprints:SOD-323F -> sc606-baseboard-footprints:D_SOD-323F; Author (none) -> Antmicro; License (none) -> Apache-2.0
- FB1: value BLM18EG221SN1D -> FB_220Z_1A_0603; footprint sc606-baseboard-footprints:0603 -> sc606-baseboard-footprints:FB_0603_1608Metric; symbol sc606-baseboard:BLM18EG221SN1D -> sc606-baseboard:FB_220Z_1A_0603; Author (none) -> Antmicro; License (none) -> Apache-2.0
- IC2: value TPS7A0518PDBVT -> TPS7A0518P_SOT23-5; symbol sc606-baseboard:TPS7A0518PDBVT -> sc606-baseboard:TPS7A0518P_SOT23-5; Author (none) -> Antmicro; License (none) -> Apache-2.0
- J6, J9: Author (none) -> Antmicro; License (none) -> Apache-2.0; Manufacturer Pulse Electronics Network -> Pulse
- L22: footprint sc606-baseboard-footprints:FIL_NFP0QHB242HS2D -> sc606-baseboard-footprints:L_Murata_025020_0605Metric; Author (none) -> Antmicro; License (none) -> Apache-2.0; Manufacturer MURATA -> Murata
- Q7: Author (none) -> Antmicro; License (none) -> Apache-2.0
- R107: footprint sc606-baseboard-footprints:0402-res -> sc606-baseboard-footprints:R_0402_1005Metric; Author (none) -> Antmicro; License (none) -> Apache-2.0; MPN CRCW040210K0FKEDHP -> CR0402-FX-1002GLF; Manufacturer VISHAY -> Bourns; Tolerance (none) -> 1%
- R108: footprint sc606-baseboard-footprints:0402-res -> sc606-baseboard-footprints:R_0402_1005Metric; Author (none) -> Antmicro; License (none) -> Apache-2.0; MPN ERJ2RKF1101X -> CR0402-FX-1101GLF; Manufacturer PANASONIC_ELECTRONIC_COMPONENTS -> Bourns; Tolerance (none) -> 1%
- R109: footprint sc606-baseboard-footprints:0402-res -> sc606-baseboard-footprints:R_0402_1005Metric; Author (none) -> Antmicro; License (none) -> Apache-2.0; MPN RC0402FR-072K2L -> CR0402-FX-2201GLF; Manufacturer YAGEO -> Bourns; Tolerance (none) -> 1%
- R110: footprint sc606-baseboard-footprints:0402-res -> sc606-baseboard-footprints:R_0402_1005Metric; Author (none) -> Antmicro; Current (none) -> 1A; License (none) -> Apache-2.0; Manufacturer PANASONIC -> Panasonic
- SW1: value 1X03 -> PinHeader_1x3_P2.54mm_Drill1.1mm; footprint sc606-baseboard-footprints:MH_1X03_2.54 -> sc606-baseboard-footprints:PinHeader_1x3_P2.54_Drill1.1mm; symbol sc606-baseboard:1X03 -> sc606-baseboard:PinHeader_1x3_P2.54mm_Drill1.1mm; Author (none) -> Antmicro; License (none) -> Apache-2.0; Manufacturer Wurth Elektronik -> Würth Elektronik
- U13: value FT232RQ-REEL -> FT232R_QFN; symbol sc606-baseboard:FT232RQ-REEL -> sc606-baseboard:FT232R_QFN; Author (none) -> Antmicro; License (none) -> Apache-2.0; Manufacturer FTDI, Future Technology Devices International Ltd -> FTDI
- U9: Author (none) -> Antmicro; License (none) -> Apache-2.0; Manufacturer ON SEMI -> ON Semiconductor
Connections:
- no-connect marks 36 -> 42
Other:
- note added: "Power flags"
- moved on the sheet: C108, C109, C110, C111, C112, C113, C114, C115, C116, C117, C142, C143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

Commit message: [#61796] Run globlib
Parts:
- C108, C109, C113, C116, C117, C142: footprint sc606-baseboard-footprints:C_0402_1005Metric -> antmicro-footprints:C_0402_1005Metric; symbol sc606-baseboard:C_100n_0402 -> antmicroCapacitors0402:C_100n_0402
- C110, C143: footprint sc606-baseboard-footprints:C_0402_1005Metric -> antmicro-footprints:C_0402_1005Metric; symbol sc606-baseboard:C_4u7_0402 -> antmicroCapacitors0402:C_4u7_0402
- C111: footprint sc606-baseboard-footprints:C_0402_1005Metric -> antmicro-footprints:C_0402_1005Metric; symbol sc606-baseboard:C_2u2_0402 -> antmicroCapacitors0402:C_2u2_0402
- C112, C114: footprint sc606-baseboard-footprints:C_0402_1005Metric -> antmicro-footprints:C_0402_1005Metric; symbol sc606-baseboard:C_47p_0402 -> antmicroCapacitors0402:C_47p_0402
- C115: footprint sc606-baseboard-footprints:C_0402_1005Metric -> antmicro-footprints:C_0402_1005Metric; symbol sc606-baseboard:C_1u_0402 -> antmicroCapacitors0402:C_1u_0402
- D20, D21, D23: footprint sc606-baseboard-footprints:Nexperia_DFN-10_2.5x1mm_P0.5mm -> antmicro-footprints:Nexperia_DFN-10_2.5x1mm_P0.5mm; symbol sc606-baseboard:PUSB3F96X_PASS -> antmicroTVSDiodes:PUSB3F96X_PASS
- D22, D43: footprint sc606-baseboard-footprints:D_SOD-323F -> antmicro-footprints:D_SOD-323F; symbol sc606-baseboard:1N4148WS -> antmicroDiodesRectifiersSingle:1N4148WS
- FB1: footprint sc606-baseboard-footprints:FB_0603_1608Metric -> antmicro-footprints:FB_0603_1608Metric; symbol sc606-baseboard:FB_220Z_1A_0603 -> antmicroFerriteBeadsandChips:FB_220Z_1A_Murata-BLM18EG_0603
- IC2: footprint sc606-baseboard-footprints:SOT-23-5 -> antmicro-footprints:SOT-23-5; symbol sc606-baseboard:TPS7A0518P_SOT23-5 -> antmicroPMICVoltageRegulatorsLinear:TPS7A0518P_SOT23-5
- J6, J9: footprint sc606-baseboard-footprints:USB-C_Female_E8124-015-01 -> antmicro-footprints:USB-C_Receptacle_PulseElectronics_E8124-015-01; symbol sc606-baseboard:E8124-015-01 -> antmicroUSBConnectors:USB-C_PulseElectronics_E8124-015-01
- L22: footprint sc606-baseboard-footprints:L_Murata_025020_0605Metric -> antmicro-footprints:Choke_025020_0605Metric; symbol sc606-baseboard:NFP0QHB242HS2D -> antmicroCommonModeChokes:Choke_NFP0QHB242HS2D
- Q7: footprint sc606-baseboard-footprints:SOT-23-3 -> antmicro-footprints:SOT-23-3; symbol sc606-baseboard:BSS138-7-F -> antmicroTransistorsFETsMOSFETsSingle:BSS138-7-F
- R107: footprint sc606-baseboard-footprints:R_0402_1005Metric -> antmicro-footprints:R_0402_1005Metric; symbol sc606-baseboard:R_10k_0402 -> antmicroResistors0402:R_10k_0402
- R108: footprint sc606-baseboard-footprints:R_0402_1005Metric -> antmicro-footprints:R_0402_1005Metric; symbol sc606-baseboard:R_1k1_0402 -> antmicroResistors0402:R_1k1_0402
- R109: footprint sc606-baseboard-footprints:R_0402_1005Metric -> antmicro-footprints:R_0402_1005Metric; symbol sc606-baseboard:R_2k2_0402 -> antmicroResistors0402:R_2k2_0402
- R110: footprint sc606-baseboard-footprints:R_0402_1005Metric -> antmicro-footprints:R_0402_1005Metric; symbol sc606-baseboard:R_0R_0402 -> antmicroResistors0402:R_0R_0402
- SW1: footprint sc606-baseboard-footprints:PinHeader_1x3_P2.54_Drill1.1mm -> antmicro-footprints:PinHeader_1x3_P2.54mm_Drill1.1mm; symbol sc606-baseboard:PinHeader_1x3_P2.54mm_Drill1.1mm -> antmicroGenericPinHeaders:PinHeader_1x3_P2.54mm_Drill1.1mm
- U13: footprint sc606-baseboard-footprints:QFN-32-1EP_5x5mm -> antmicro-footprints:QFN-32-1EP_5x5mm; symbol sc606-baseboard:FT232R_QFN -> antmicroInterfaceControllers:FT232R_QFN
- U9: footprint sc606-baseboard-footprints:MSOP-10_W3mm -> antmicro-footprints:MSOP-10_W3mm; symbol sc606-baseboard:FSUSB30MUX -> antmicroInterfaceAnalogSwitchesSpecialPurpose:FSUSB30MUX

Commit message: [#61796] Update schematics
Parts:
- C112, C114: MPN GRM1555C1E470JA01D -> C0402C470J5GACTU; Manufacturer Murata -> KEMET
- FB1: value FB_220Z_1A_0603 -> FB_220Z_1A_Murata-BLM18EG_0603; Val (none) -> 220Z/1A
- J6, J9: value E8124-015-01 -> USB-C_PulseElectronics_E8124-015-01; Manufacturer Pulse -> Pulse Electronics
- L22: value NFP0QHB242HS2D -> Choke_NFP0QHB242HS2D; IMax (none) -> 0.1 A
- U13: Manufacturer FTDI -> FTDI Chip
Connections:
- net 5V0_DBG: now also D22.1 (C); no longer D22.K
- net 5V0_SYS: now also D22.2 (A); no longer D22.A
- net USB_FLASH_5V0: now also D43.2 (A); no longer D43.A
- net USB_VBUS_DET: now also D43.1 (C); no longer D43.K
Other:
- company: (none) -> Antmicro Ltd
- moved on the sheet: D20

Commit message: [#61796] Update designators
Parts:
- renumbered SW1 to J18
Changed lines of the file:
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@@
   (symbol (lib_id "antmicroGenericPinHeaders:PinHeader_1x3_P2.54mm_Drill1.1mm") (at 365.76 104.14 0) (unit 1)
     (in_bom yes) (on_board yes) (dnp no) (fields_autoplaced)
-    (property "Reference" "SW1" (at 372.11 105.41 0)
+    (property "Reference" "J18" (at 372.11 105.41 0)
       (effects (font (size 1.27 1.27) (thickness 0.15)) (justify left))
     )
@@
       (project "sc606-baseboard"
         (path "/d033de6c-b5da-4924-ae5b-c5bab6f8ca2c/00000000-0000-0000-0000-000061f60810"
-          (reference "SW1") (unit 1)
+          (reference "J18") (unit 1)
         )
       )
